File: Motherboard/ANALOG_EXPANSION.sch (KiCad schematic (older format))
At the start: 43 parts

Commit message: - Refer to Google Drive BOM for list of changes for v1.1 - Create drawing for Hella BLDC controller plate.
Parts:
- AI30-35_CONN1, AI36-41_CONN1, AI42-47_CONN1: footprint Smart_Tank:PHX_TB_HDR_10_POS_(1757323) -> Smart_Tank:PHX_TB_HDR_10_POS_STR_(1755817)
Changed lines of the file:
@@
 3.3VDC
 $Comp
-L GND #PWR010
+L GND #PWR011
 U 1 1 57920B33
 P 1900 2600
-F 0 "#PWR010" H 1900 2350 50  0001 C CNN
+F 0 "#PWR011" H 1900 2350 50  0001 C CNN
 F 1 "GND" H 1900 2450 50  0000 C CNN
 F 2 "" H 1900 2600 50  0000 C CNN
@@
 3.3VDC
 $Comp
-L GND #PWR011
+L GND #PWR012
 U 1 1 57922DF1
 P 4550 2600
-F 0 "#PWR011" H 4550 2350 50  0001 C CNN
+F 0 "#PWR012" H 4550 2350 50  0001 C CNN
 F 1 "GND" H 4550 2450 50  0000 C CNN
 F 2 "" H 4550 2600 50  0000 C CNN
@@
 3.3VDC
 $Comp
-L GND #PWR012
+L GND #PWR013
 U 1 1 57923753
 P 7200 2650
-F 0 "#PWR012" H 7200 2400 50  0001 C CNN
+F 0 "#PWR013" H 7200 2400 50  0001 C CNN
 F 1 "GND" H 7200 2500 50  0000 C CNN
 F 2 "" H 7200 2650 50  0000 C CNN
@@
 3.3VDC
 $Comp
-L GND #PWR013
+L GND #PWR014
 U 1 1 579237E1
 P 9850 2650
-F 0 "#PWR013" H 9850 2400 50  0001 C CNN
+F 0 "#PWR014" H 9850 2400 50  0001 C CNN
 F 1 "GND" H 9850 2500 50  0000 C CNN
 F 2 "" H 9850 2650 50  0000 C CNN
@@
 F 0 "AI30-35_CONN1" H 1100 4500 50  0000 C CNN
 F 1 "CONN_01X10" H 1100 5650 50  0000 C CNN
-F 2 "Smart_Tank:PHX_TB_HDR_10_POS_(1757323)" H 1100 5100 50  0001 C CNN
+F 2 "Smart_Tank:PHX_TB_HDR_10_POS_STR_(1755817)" H 1100 5100 50  0001 C CNN
 F 3 "" H 1100 5100 50  0000 C CNN
 	1    1100 5100
@@
 PWR
 $Comp
-L GND #PWR014
+L GND #PWR015
 U 1 1 5797F880
 P 1750 5600
-F 0 "#PWR014" H 1750 5350 50  0001 C CNN
+F 0 "#PWR015" H 1750 5350 50  0001 C CNN
 F 1 "GND" H 1750 5450 50  0000 C CNN
 F 2 "" H 1750 5600 50  0000 C CNN
@@
 24VDC
 $Comp
-L GND #PWR015
+L GND #PWR016
 U 1 1 579F7225
 P 3700 5250
-F 0 "#PWR015" H 3700 5000 50  0001 C CNN
+F 0 "#PWR016" H 3700 5000 50  0001 C CNN
 F 1 "GND" H 3700 5100 50  0000 C CNN
 F 2 "" H 3700 5250 50  0000 C CNN
@@
 F 0 "AI36-41_CONN1" H 4650 4500 50  0000 C CNN
 F 1 "CONN_01X10" H 4650 5650 50  0000 C CNN
-F 2 "Smart_Tank:PHX_TB_HDR_10_POS_(1757323)" H 4650 5100 50  0001 C CNN
+F 2 "Smart_Tank:PHX_TB_HDR_10_POS_STR_(1755817)" H 4650 5100 50  0001 C CNN
 F 3 "" H 4650 5100 50  0000 C CNN
 	1    4650 5100
@@
 PWR
 $Comp
-L GND #PWR016
+L GND #PWR017
 U 1 1 57AA6E5B
 P 5300 5600
-F 0 "#PWR016" H 5300 5350 50  0001 C CNN
+F 0 "#PWR017" H 5300 5350 50  0001 C CNN
 F 1 "GND" H 5300 5450 50  0000 C CNN
 F 2 "" H 5300 5600 50  0000 C CNN
@@
 F 0 "AI42-47_CONN1" H 8150 4500 50  0000 C CNN
 F 1 "CONN_01X10" H 8150 5650 50  0000 C CNN
-F 2 "Smart_Tank:PHX_TB_HDR_10_POS_(1757323)" H 8150 5100 50  0001 C CNN
+F 2 "Smart_Tank:PHX_TB_HDR_10_POS_STR_(1755817)" H 8150 5100 50  0001 C CNN
 F 3 "" H 8150 5100 50  0000 C CNN
 	1    8150 5100
@@
 PWR
 $Comp
-L GND #PWR017
+L GND #PWR018
 U 1 1 57AA7154
 P 8800 5600
-F 0 "#PWR017" H 8800 5350 50  0001 C CNN
+F 0 "#PWR018" H 8800 5350 50  0001 C CNN
 F 1 "GND" H 8800 5450 50  0000 C CNN
 F 2 "" H 8800 5600 50  0000 C CNN
@@
 Connection ~ 8950 4650
 $Comp
-L GND #PWR018
+L GND #PWR019
 U 1 1 57AA9513
 P 7250 5250
-F 0 "#PWR018" H 7250 5000 50  0001 C CNN
+F 0 "#PWR019" H 7250 5000 50  0001 C CNN
 F 1 "GND" H 7250 5100 50  0000 C CNN
 F 2 "" H 7250 5250 50  0000 C CNN
@@
 Connection ~ 7250 5150
 $Comp
-L GND #PWR019
+L GND #PWR020
 U 1 1 57AA9683
 P 10750 5250
-F 0 "#PWR019" H 10750 5000 50  0001 C CNN
+F 0 "#PWR020" H 10750 5000 50  0001 C CNN
 F 1 "GND" H 10750 5100 50  0000 C CNN
 F 2 "" H 10750 5250 50  0000 C CNN

Commit message: - Created Modbus Adapter.
Parts:
- ADC_AI16-23, ADC_AI24-31, ADC_AI32-39, ADC_AI40-47: symbol TI_ADC_(ADS8332) -> Smart-Tank-Motherboard-rescue:TI_ADC_(ADS8332)
- AI30-35_CONN1, AI36-41_CONN1, AI42-47_CONN1: symbol CONN_01X10 -> Smart-Tank-Motherboard-rescue:CONN_01X10
- C1, C10, C11, C12, C2, C3, C4, C5, C6, C7, C8, C9: symbol C -> Smart-Tank-Motherboard-rescue:C
- INPUT_SEL_1, INPUT_SEL_2, INPUT_SEL_3: symbol CTS_DIP_SW_(219-6MST) -> Smart-Tank-Motherboard-rescue:CTS_DIP_SW_(219-6MST)
- PWR_SEL_1, PWR_SEL_2, PWR_SEL_3: symbol CONN_01X03 -> Smart-Tank-Motherboard-rescue:CONN_01X03
- R20, R21, R22, R23, R24, R25, R26, R27, R28, R29, R30, R31, R32, R33, R34, R35, R36, R37: symbol R -> Smart-Tank-Motherboard-rescue:R
Changed lines of the file:
@@
-EESchema Schematic File Version 2
-LIBS:Smart Tank Motherboard-rescue
-LIBS:power
-LIBS:device
-LIBS:transistors
-LIBS:conn
-LIBS:linear
-LIBS:regul
-LIBS:74xx
-LIBS:cmos4000
-LIBS:adc-dac
-LIBS:memory
-LIBS:xilinx
-LIBS:microcontrollers
-LIBS:dsp
-LIBS:microchip
-LIBS:analog_switches
-LIBS:motorola
-LIBS:texas
-LIBS:intel
-LIBS:audio
-LIBS:interface
-LIBS:digital-audio
-LIBS:philips
-LIBS:display
-LIBS:cypress
-LIBS:siliconi
-LIBS:opto
-LIBS:atmel
-LIBS:contrib
-LIBS:valves
+EESchema Schematic File Version 4
 LIBS:Smart Tank Motherboard-cache
-EELAYER 25 0
+EELAYER 29 0
 EELAYER END
 $Descr A4 11693 8268
@@
 $EndDescr
 $Comp
-L TI_ADC_(ADS8332) ADC_AI16-23
+L Smart-Tank-Motherboard-rescue:TI_ADC_(ADS8332) ADC_AI16-23
 U 1 1 57920A54
 P 1350 2000
@@
 3.3VDC
 $Comp
-L GND #PWR011
+L Smart-Tank-Motherboard-rescue:GND #PWR011
 U 1 1 57920B33
 P 1900 2600
@@
 3.3VDC
 $Comp
-L C C3
+L Smart-Tank-Motherboard-rescue:C C3
 U 1 1 57920B72
 P 2450 2450
@@
 $EndComp
 $Comp
-L C C2
+L Smart-Tank-Motherboard-rescue:C C2
 U 1 1 57920D8A
 P 2450 1950
@@
 $EndComp
 $Comp
-L C C1
+L Smart-Tank-Motherboard-rescue:C C1
 U 1 1 57920DB3
 P 2450 1650
@@
 AI_CONVST
 $Comp
-L TI_ADC_(ADS8332) ADC_AI24-31
+L Smart-Tank-Motherboard-rescue:TI_ADC_(ADS8332) ADC_AI24-31
 U 1 1 57922DE2
 P 4000 2000
@@
 3.3VDC
 $Comp
-L GND #PWR012
+L Smart-Tank-Motherboard-rescue:GND #PWR012
 U 1 1 57922DF1
 P 4550 2600
@@
 3.3VDC
 $Comp
-L C C9
+L Smart-Tank-Motherboard-rescue:C C9
 U 1 1 57922DF8
 P 5100 2450
@@
 $EndComp
 $Comp
-L C C8
+L Smart-Tank-Motherboard-rescue:C C8
 U 1 1 57922DFE
 P 5100 1950
@@
 $EndComp
 $Comp
-L C C7
+L Smart-Tank-Motherboard-rescue:C C7
 U 1 1 57922E04
 P 5100 1650
@@
 AI_CONVST
 $Comp
-L TI_ADC_(ADS8332) ADC_AI32-39
+L Smart-Tank-Motherboard-rescue:TI_ADC_(ADS8332) ADC_AI32-39
 U 1 1 57923744
 P 6650 2000
@@
 3.3VDC
 $Comp
-L GND #PWR013
+L Smart-Tank-Motherboard-rescue:GND #PWR013
 U 1 1 57923753
 P 7200 2650
@@
 3.3VDC
 $Comp
-L C C6
+L Smart-Tank-Motherboard-rescue:C C6
 U 1 1 5792375A
 P 7750 2450
@@
 $EndComp
 $Comp
-L C C5
+L Smart-Tank-Motherboard-rescue:C C5
 U 1 1 57923760
 P 7750 1950
@@
 $EndComp
 $Comp
-L C C4
+L Smart-Tank-Motherboard-rescue:C C4
 U 1 1 57923766
 P 7750 1650
@@
 AI_CONVST
 $Comp
-L TI_ADC_(ADS8332) ADC_AI40-47
+L Smart-Tank-Motherboard-rescue:TI_ADC_(ADS8332) ADC_AI40-47
 U 1 1 579237D2
 P 9300 2000
@@
 3.3VDC
 $Comp
-L GND #PWR014
+L Smart-Tank-Motherboard-rescue:GND #PWR014
 U 1 1 579237E1
 P 9850 2650
@@
 3.3VDC
 $Comp
-L C C12
+L Smart-Tank-Motherboard-rescue:C C12
 U 1 1 579237E8
 P 10400 2450
@@
 $EndComp
 $Comp
-L C C11
+L Smart-Tank-Motherboard-rescue:C C11
 U 1 1 579237EE
 P 10400 1950
@@
 $EndComp
 $Comp
-L C C10
+L Smart-Tank-Motherboard-rescue:C C10
 U 1 1 579237F4
 P 10400 1650
@@
 AI_CONVST
 $Comp
-L CONN_01X10 AI30-35_CONN1
+L Smart-Tank-Motherboard-rescue:CONN_01X10 AI30-35_CONN1
 U 1 1 5797F86F
 P 1100 5100
@@
 PWR
 $Comp
-L GND #PWR015
+L Smart-Tank-Motherboard-rescue:GND #PWR015
 U 1 1 5797F880
 P 1750 5600
@@
 $EndComp
 $Comp
-L CONN_01X03 PWR_SEL_1
+L Smart-Tank-Motherboard-rescue:CONN_01X03 PWR_SEL_1
 U 1 1 5797F886
 P 1100 4050
@@
 24VDC
 $Comp
-L GND #PWR016
+L Smart-Tank-Motherboard-rescue:GND #PWR016
 U 1 1 579F7225
 P 3700 5250
@@
 $EndComp
 $Comp
-L CTS_DIP_SW_(219-6MST) INPUT_SEL_1
+L Smart-Tank-Motherboard-rescue:CTS_DIP_SW_(219-6MST) INPUT_SEL_1
 U 1 1 579F722B
 P 2850 4900
@@
 $EndComp
 $Comp
-L R R26
+L Smart-Tank-Motherboard-rescue:R R26
 U 1 1 57A153EA
 P 3350 4650
@@
 $EndComp
 $Comp
-L R R27
+L Smart-Tank-Motherboard-rescue:R R27
 U 1 1 57A153F0
 P 3350 4750
@@
 $EndComp
 $Comp
-L R R28
+L Smart-Tank-Motherboard-rescue:R R28
 U 1 1 57A153F6
 P 3350 4850
@@
 $EndComp
 $Comp
-L R R29
+L Smart-Tank-Motherboard-rescue:R R29
 U 1 1 57A153FC
 P 3350 4950
@@
 $EndComp
 $Comp
-L R R30
+L Smart-Tank-Motherboard-rescue:R R30
 U 1 1 57A15402
 P 3350 5050
@@
 $EndComp
 $Comp
-L R R31
+L Smart-Tank-Motherboard-rescue:R R31
 U 1 1 57A15408
 P 3350 5150
@@
 Connection ~ 1900 4650
 $Comp
-L CONN_01X10 AI36-41_CONN1
+L Smart-Tank-Motherboard-rescue:CONN_01X10 AI36-41_CONN1
 U 1 1 57AA6E4A
 P 4650 5100
@@
 PWR
 $Comp
-L GND #PWR017
+L Smart-Tank-Motherboard-rescue:GND #PWR017
 U 1 1 57AA6E5B
 P 5300 5600
@@
 $EndComp
 $Comp
-L CONN_01X03 PWR_SEL_2
+L Smart-Tank-Motherboard-rescue:CONN_01X03 PWR_SEL_2
 U 1 1 57AA6E61
 P 4650 4050
@@
 24VDC
 $Comp
-L CTS_DIP_SW_(219-6MST) INPUT_SEL_2
+L Smart-Tank-Motherboard-rescue:CTS_DIP_SW_(219-6MST) INPUT_SEL_2
 U 1 1 57AA6E70
 P 6400 4900
@@
 Connection ~ 5450 4650
 $Comp
-L CONN_01X10 AI42-47_CONN1
+L Smart-Tank-Motherboard-rescue:CONN_01X10 AI42-47_CONN1
 U 1 1 57AA7143
 P 8150 5100
@@
 PWR
 $Comp
-L GND #PWR018
+L Smart-Tank-Motherboard-rescue:GND #PWR018
 U 1 1 57AA7154
 P 8800 5600
@@
 $EndComp
 $Comp
-L CONN_01X03 PWR_SEL_3
+L Smart-Tank-Motherboard-rescue:CONN_01X03 PWR_SEL_3
 U 1 1 57AA715A
 P 8150 4050
@@
 24VDC
 $Comp
-L CTS_DIP_SW_(219-6MST) INPUT_SEL_3
+L Smart-Tank-Motherboard-rescue:CTS_DIP_SW_(219-6MST) INPUT_SEL_3
 U 1 1 57AA7169
 P 9900 4900
@@
 Connection ~ 8950 4650
 $Comp
-L GND #PWR019
+L Smart-Tank-Motherboard-rescue:GND #PWR019
 U 1 1 57AA9513
 P 7250 5250
@@
 $EndComp
 $Comp
-L R R20
+L Smart-Tank-Motherboard-rescue:R R20
 U 1 1 57AA9519
 P 6900 4650
@@
 $EndComp
 $Comp
-L R R21
+L Smart-Tank-Motherboard-rescue:R R21
 U 1 1 57AA9520
 P 6900 4750
@@
 $EndComp
 $Comp
-L R R22
+L Smart-Tank-Motherboard-rescue:R R22
 U 1 1 57AA9527
 P 6900 4850
@@
 $EndComp
 $Comp
-L R R23
+L Smart-Tank-Motherboard-rescue:R R23
 U 1 1 57AA952E
 P 6900 4950
@@
 $EndComp
 $Comp
-L R R24
+L Smart-Tank-Motherboard-rescue:R R24
 U 1 1 57AA9535
 P 6900 5050
@@
 $EndComp
 $Comp
-L R R25
+L Smart-Tank-Motherboard-rescue:R R25
 U 1 1 57AA953C
 P 6900 5150
@@
 Connection ~ 7250 5150
 $Comp
-L GND #PWR020
+L Smart-Tank-Motherboard-rescue:GND #PWR020
 U 1 1 57AA9683
 P 10750 5250
@@
 $EndComp
 $Comp
-L R R32
+L Smart-Tank-Motherboard-rescue:R R32
 U 1 1 57AA9689
 P 10400 4650
@@
 $EndComp
 $Comp
-L R R33
+L Smart-Tank-Motherboard-rescue:R R33
 U 1 1 57AA9690
 P 10400 4750
@@
 $EndComp
 $Comp
-L R R34
+L Smart-Tank-Motherboard-rescue:R R34
 U 1 1 57AA9697
 P 10400 4850
@@
 $EndComp
 $Comp
-L R R35
+L Smart-Tank-Motherboard-rescue:R R35
 U 1 1 57AA969E
 P 10400 4950
@@
 $EndComp
 $Comp
-L R R36
+L Smart-Tank-Motherboard-rescue:R R36
 U 1 1 57AA96A5
 P 10400 5050
@@
 $EndComp
 $Comp
-L R R37
+L Smart-Tank-Motherboard-rescue:R R37
 U 1 1 57AA96AC
 P 10400 5150
