File: Motherboard/TC_INPUTS.sch (KiCad schematic (older format))
At the start: 19 parts

Commit message: - Refer to Google Drive BOM for list of changes for v1.1 - Create drawing for Hella BLDC controller plate.
Parts:
- TC_INPUTS1: footprint Smart_Tank:PHX_TB_HDR_4_POS_(1757268) -> Smart_Tank:PHX_TB_HDR_4_POS_STR_(1755752)
Changed lines of the file:
@@
 F 0 "TC_INPUTS1" H 2850 1500 50  0000 C CNN
 F 1 "CONN_01X04" H 2850 950 50  0000 C CNN
-F 2 "Smart_Tank:PHX_TB_HDR_4_POS_(1757268)" H 2850 1200 50  0001 C CNN
+F 2 "Smart_Tank:PHX_TB_HDR_4_POS_STR_(1755752)" H 2850 1200 50  0001 C CNN
 F 3 "" H 2850 1200 50  0000 C CNN
 	1    2850 1200
@@
 Connection ~ 7250 2550
 $Comp
-L GND #PWR020
+L GND #PWR021
 U 1 1 5797493B
 P 4600 3400
-F 0 "#PWR020" H 4600 3150 50  0001 C CNN
+F 0 "#PWR021" H 4600 3150 50  0001 C CNN
 F 1 "GND" H 4600 3250 50  0000 C CNN
 F 2 "" H 4600 3400 50  0000 C CNN
@@
 Connection ~ 7250 5350
 $Comp
-L GND #PWR021
+L GND #PWR022
 U 1 1 579754CE
 P 4600 6200
-F 0 "#PWR021" H 4600 5950 50  0001 C CNN
+F 0 "#PWR022" H 4600 5950 50  0001 C CNN
 F 1 "GND" H 4600 6050 50  0000 C CNN
 F 2 "" H 4600 6200 50  0000 C CNN

Commit message: - Created Modbus Adapter.
Parts:
- C14, C16, C17, C18, C19, C22, C23, C24, C25, C26: symbol C -> Smart-Tank-Motherboard-rescue:C
- R14, R15, R16, R44, R45, R46: symbol R -> Smart-Tank-Motherboard-rescue:R
- TC_INPUTS1: symbol CONN_01X04 -> Smart-Tank-Motherboard-rescue:CONN_01X04
- TEMP_1, TEMP_2: symbol TEMP_COND_(AD8497) -> Smart-Tank-Motherboard-rescue:TEMP_COND_(AD8497)
Changed lines of the file:
@@
-EESchema Schematic File Version 2
-LIBS:Smart Tank Motherboard-rescue
-LIBS:power
-LIBS:device
-LIBS:transistors
-LIBS:conn
-LIBS:linear
-LIBS:regul
-LIBS:74xx
-LIBS:cmos4000
-LIBS:adc-dac
-LIBS:memory
-LIBS:xilinx
-LIBS:microcontrollers
-LIBS:dsp
-LIBS:microchip
-LIBS:analog_switches
-LIBS:motorola
-LIBS:texas
-LIBS:intel
-LIBS:audio
-LIBS:interface
-LIBS:digital-audio
-LIBS:philips
-LIBS:display
-LIBS:cypress
-LIBS:siliconi
-LIBS:opto
-LIBS:atmel
-LIBS:contrib
-LIBS:valves
+EESchema Schematic File Version 4
 LIBS:Smart Tank Motherboard-cache
-EELAYER 25 0
+EELAYER 29 0
 EELAYER END
 $Descr A4 11693 8268
@@
 $EndDescr
 $Comp
-L TEMP_COND_(AD8497) TEMP_1
+L Smart-Tank-Motherboard-rescue:TEMP_COND_(AD8497) TEMP_1
 U 1 1 57968DB6
 P 6000 2600
@@
 $EndComp
 $Comp
-L CONN_01X04 TC_INPUTS1
+L Smart-Tank-Motherboard-rescue:CONN_01X04 TC_INPUTS1
 U 1 1 57968E7F
 P 2850 1200
@@
 -TEMP_2
 $Comp
-L C C16
+L Smart-Tank-Motherboard-rescue:C C16
 U 1 1 5796911E
 P 6000 2050
@@
 	6550 2450 6350 2450
 $Comp
-L R R15
+L Smart-Tank-Motherboard-rescue:R R15
 U 1 1 57969213
 P 5450 1700
@@
 $EndComp
 $Comp
-L R R16
+L Smart-Tank-Motherboard-rescue:R R16
 U 1 1 579692D0
 P 6550 1700
@@
 Connection ~ 6550 2050
 $Comp
-L R R14
+L Smart-Tank-Motherboard-rescue:R R14
 U 1 1 57969336
 P 5000 1450
@@
 	5450 1150 5450 1550
 $Comp
-L C C14
+L Smart-Tank-Motherboard-rescue:C C14
 U 1 1 579693DF
 P 5000 2050
@@
 $EndComp
 $Comp
-L C C18
+L Smart-Tank-Motherboard-rescue:C C18
 U 1 1 579694AA
 P 6950 2050
@@
 3.3VDC
 $Comp
-L C C17
+L Smart-Tank-Motherboard-rescue:C C17
 U 1 1 5797473E
 P 6850 2900
@@
 $EndComp
 $Comp
-L C C19
+L Smart-Tank-Motherboard-rescue:C C19
 U 1 1 57974774
 P 7250 2900
@@
 Connection ~ 7250 2550
 $Comp
-L GND #PWR021
+L Smart-Tank-Motherboard-rescue:GND #PWR021
 U 1 1 5797493B
 P 4600 3400
@@
 Connection ~ 6400 2750
 $Comp
-L TEMP_COND_(AD8497) TEMP_2
+L Smart-Tank-Motherboard-rescue:TEMP_COND_(AD8497) TEMP_2
 U 1 1 57975477
 P 6000 5400
@@
 $EndComp
 $Comp
-L C C23
+L Smart-Tank-Motherboard-rescue:C C23
 U 1 1 5797547E
 P 6000 4850
@@
 	6550 5250 6350 5250
 $Comp
-L R R45
+L Smart-Tank-Motherboard-rescue:R R45
 U 1 1 5797548B
 P 5450 4500
@@
 $EndComp
 $Comp
-L R R46
+L Smart-Tank-Motherboard-rescue:R R46
 U 1 1 57975492
 P 6550 4500
@@
 Connection ~ 6550 4850
 $Comp
-L R R44
+L Smart-Tank-Motherboard-rescue:R R44
 U 1 1 5797549B
 P 5000 4250
@@
 	5450 3950 5450 4350
 $Comp
-L C C22
+L Smart-Tank-Motherboard-rescue:C C22
 U 1 1 579754A4
 P 5000 4850
@@
 $EndComp
 $Comp
-L C C25
+L Smart-Tank-Motherboard-rescue:C C25
 U 1 1 579754AB
 P 6950 4850
@@
 3.3VDC
 $Comp
-L C C24
+L Smart-Tank-Motherboard-rescue:C C24
 U 1 1 579754BC
 P 6850 5700
@@
 $EndComp
 $Comp
-L C C26
+L Smart-Tank-Motherboard-rescue:C C26
 U 1 1 579754C3
 P 7250 5700
@@
 Connection ~ 7250 5350
 $Comp
-L GND #PWR022
+L Smart-Tank-Motherboard-rescue:GND #PWR022
 U 1 1 579754CE
 P 4600 6200
