File: Motherboard/Smart Tank Motherboard.sch (KiCad schematic (older format))
At the start: 18 parts, among them Q5 MOSFET_N_(2N7002P,215), Q6 MOSFET_N_(2N7002P,215), Q7 MOSFET_N_(2N7002P,215)

Commit message: - Refer to Google Drive BOM for list of changes for v1.1 - Create drawing for Hella BLDC controller plate.
Parts:
- GPIO_CONN1: footprint Smart_Tank:PHX_TB_HDR_10_POS_(1757323) -> Smart_Tank:PHX_TB_HDR_10_POS_STR_(1755817)
- PWR_CONN1: footprint Smart_Tank:PHX_TB_HDR_4_POS_(1757268) -> Smart_Tank:PHX_TB_HDR_4_POS_STR_(1755752)
Changed lines of the file:
@@
 F 0 "PWR_CONN1" H 1850 2550 50  0000 C CNN
 F 1 "CONN_01X04" H 1850 2050 50  0000 C CNN
-F 2 "Smart_Tank:PHX_TB_HDR_4_POS_(1757268)" H 1850 2300 50  0001 C CNN
+F 2 "Smart_Tank:PHX_TB_HDR_4_POS_STR_(1755752)" H 1850 2300 50  0001 C CNN
 F 3 "" H 1850 2300 50  0000 C CNN
 	1    1850 2300
@@
 F 0 "GPIO_CONN1" H 1850 5800 50  0000 C CNN
 F 1 "CONN_01X10" H 1850 4700 50  0000 C CNN
-F 2 "Smart_Tank:PHX_TB_HDR_10_POS_(1757323)" H 1850 5250 50  0001 C CNN
+F 2 "Smart_Tank:PHX_TB_HDR_10_POS_STR_(1755817)" H 1850 5250 50  0001 C CNN
 F 3 "" H 1850 5250 50  0000 C CNN
 	1    1850 5250

Commit message: - Created Modbus Adapter.
Parts:
- 24VDC_FUSE1: symbol FUSE_HOLDER_(01220083Z) -> Smart-Tank-Motherboard-rescue:FUSE_HOLDER_(01220083Z)
- D2, D3, D4: symbol DIODE_(1N4148X-TP) -> Smart-Tank-Motherboard-rescue:DIODE_(1N4148X-TP)
- E-STOP_RLY1, RELAY_1, RELAY_2: symbol OMRON_RELAY_(G6L-1F-DC24) -> Smart-Tank-Motherboard-rescue:OMRON_RELAY_(G6L-1F-DC24)
- GPIO_CONN1: symbol CONN_01X10 -> Smart-Tank-Motherboard-rescue:CONN_01X10
- PWR_CONN1: symbol CONN_01X04 -> Smart-Tank-Motherboard-rescue:CONN_01X04
- Q5, Q6, Q7: symbol MOSFET_N_(2N7002P,215) -> Smart-Tank-Motherboard-rescue:MOSFET_N_(2N7002P,215)
- R10, R11, R12, R13, R8, R9: symbol R -> Smart-Tank-Motherboard-rescue:R
Changed lines of the file:
@@
-EESchema Schematic File Version 2
-LIBS:Smart Tank Motherboard-rescue
-LIBS:power
-LIBS:device
-LIBS:transistors
-LIBS:conn
-LIBS:linear
-LIBS:regul
-LIBS:74xx
-LIBS:cmos4000
-LIBS:adc-dac
-LIBS:memory
-LIBS:xilinx
-LIBS:microcontrollers
-LIBS:dsp
-LIBS:microchip
-LIBS:analog_switches
-LIBS:motorola
-LIBS:texas
-LIBS:intel
-LIBS:audio
-LIBS:interface
-LIBS:digital-audio
-LIBS:philips
-LIBS:display
-LIBS:cypress
-LIBS:siliconi
-LIBS:opto
-LIBS:atmel
-LIBS:contrib
-LIBS:valves
+EESchema Schematic File Version 4
 LIBS:Smart Tank Motherboard-cache
-EELAYER 25 0
+EELAYER 29 0
 EELAYER END
 $Descr A4 11693 8268
@@
 E-STOP_OUT
 $Comp
-L GND #PWR01
+L Smart-Tank-Motherboard-rescue:GND #PWR01
 U 1 1 578941DC
 P 6950 3900
@@
 $EndSheet
 $Comp
-L FUSE_HOLDER_(01220083Z) 24VDC_FUSE1
+L Smart-Tank-Motherboard-rescue:FUSE_HOLDER_(01220083Z) 24VDC_FUSE1
 U 1 1 5790EBB7
 P 7600 2150
@@
 DIO25
 $Comp
-L OMRON_RELAY_(G6L-1F-DC24) RELAY_1
+L Smart-Tank-Motherboard-rescue:OMRON_RELAY_(G6L-1F-DC24) RELAY_1
 U 1 1 57911942
 P 5250 5000
@@
 $EndComp
 $Comp
-L MOSFET_N_(2N7002P,215) Q6
+L Smart-Tank-Motherboard-rescue:MOSFET_N_(2N7002P,215) Q6
 U 1 1 57911949
 P 4500 5350
@@
 $EndComp
 $Comp
-L R R12
+L Smart-Tank-Motherboard-rescue:R R12
 U 1 1 57911950
 P 4050 5400
@@
 $EndComp
 $Comp
-L R R9
+L Smart-Tank-Motherboard-rescue:R R9
 U 1 1 57911957
 P 3700 5550
@@
 24VDC
 $Comp
-L DIODE_(1N4148X-TP) D3
+L Smart-Tank-Motherboard-rescue:DIODE_(1N4148X-TP) D3
 U 1 1 57911960
 P 4100 5000
@@
 $EndComp
 $Comp
-L OMRON_RELAY_(G6L-1F-DC24) RELAY_2
+L Smart-Tank-Motherboard-rescue:OMRON_RELAY_(G6L-1F-DC24) RELAY_2
 U 1 1 57911F1A
 P 5250 6200
@@
 $EndComp
 $Comp
-L MOSFET_N_(2N7002P,215) Q7
+L Smart-Tank-Motherboard-rescue:MOSFET_N_(2N7002P,215) Q7
 U 1 1 57911F21
 P 4500 6550
@@
 $EndComp
 $Comp
-L R R13
+L Smart-Tank-Motherboard-rescue:R R13
 U 1 1 57911F28
 P 4050 6600
@@
 $EndComp
 $Comp
-L R R10
+L Smart-Tank-Motherboard-rescue:R R10
 U 1 1 57911F2F
 P 3700 6750
@@
 24VDC
 $Comp
-L DIODE_(1N4148X-TP) D4
+L Smart-Tank-Motherboard-rescue:DIODE_(1N4148X-TP) D4
 U 1 1 57911F38
 P 4100 6200
@@
 $EndComp
 $Comp
-L GND #PWR02
+L Smart-Tank-Motherboard-rescue:GND #PWR02
 U 1 1 579120A4
 P 3000 7000
@@
 $EndComp
 $Comp
-L OMRON_RELAY_(G6L-1F-DC24) E-STOP_RLY1
+L Smart-Tank-Motherboard-rescue:OMRON_RELAY_(G6L-1F-DC24) E-STOP_RLY1
 U 1 1 57914B8C
 P 5250 3050
@@
 $EndComp
 $Comp
-L MOSFET_N_(2N7002P,215) Q5
+L Smart-Tank-Motherboard-rescue:MOSFET_N_(2N7002P,215) Q5
 U 1 1 57914B93
 P 4500 3400
@@
 $EndComp
 $Comp
-L R R11
+L Smart-Tank-Motherboard-rescue:R R11
 U 1 1 57914B9A
 P 4050 3450
@@
 $EndComp
 $Comp
-L R R8
+L Smart-Tank-Motherboard-rescue:R R8
 U 1 1 57914BA1
 P 3700 3600
@@
 24VDC
 $Comp
-L DIODE_(1N4148X-TP) D2
+L Smart-Tank-Motherboard-rescue:DIODE_(1N4148X-TP) D2
 U 1 1 57914BAA
 P 4100 3050
@@
 $EndComp
 $Comp
-L CONN_01X04 PWR_CONN1
+L Smart-Tank-Motherboard-rescue:CONN_01X04 PWR_CONN1
 U 1 1 5791597C
 P 1850 2300
@@
 $EndSheet
 $Comp
-L CONN_01X10 GPIO_CONN1
+L Smart-Tank-Motherboard-rescue:CONN_01X10 GPIO_CONN1
 U 1 1 57988021
 P 1850 5250
@@
 	2050 2250 6950 2250
 Wire Wire Line
-	6950 2250 6950 3900
+	6950 2250 6950 3750
 Wire Wire Line
 	2050 2150 7350 2150
@@
 	2050 4800 5000 4800
 Wire Wire Line
-	4250 5000 5000 5000
+	4250 5000 4600 5000
 Wire Wire Line
 	4600 5700 4600 5550
 Wire Wire Line
-	3550 5400 3900 5400
+	3550 5400 3700 5400
 Wire Wire Line
 	4200 5400 4300 5400
@@
 	4600 5000 4600 5150
 Wire Wire Line
-	3550 4900 5000 4900
+	3550 4900 3850 4900
 Connection ~ 4600 5000
 Wire Wire Line
@@
 Connection ~ 3850 4900
 Wire Wire Line
-	4250 6200 5000 6200
+	4250 6200 4600 6200
 Wire Wire Line
 	4600 6900 4600 6750
 Wire Wire Line
-	3550 6600 3900 6600
+	3550 6600 3700 6600
 Wire Wire Line
 	4200 6600 4300 6600
@@
 	4600 6200 4600 6350
 Wire Wire Line
-	3550 6100 5000 6100
+	3550 6100 3850 6100
 Connection ~ 4600 6200
 Wire Wire Line
@@
 	2650 5000 2650 6000
 Wire Wire Line
-	3000 5700 3000 7000
+	3000 5700 3000 6900
 Connection ~ 3000 6900
 Wire Wire Line
@@
 	2550 5100 2050 5100
 Wire Wire Line
-	4250 3050 5000 3050
+	4250 3050 4600 3050
 Wire Wire Line
 	4600 3600 4600 3750
 Wire Wire Line
-	3550 3450 3900 3450
+	3550 3450 3700 3450
 Wire Wire Line
 	4200 3450 4300 3450
@@
 	4600 3050 4600 3200
 Wire Wire Line
-	3550 2950 5000 2950
+	3550 2950 3850 2950
 Connection ~ 4600 3050
 Wire Wire Line
@@
 	2050 5700 2250 5700
 Wire Wire Line
-	2250 5600 2250 6900
+	2250 5600 2250 5700
 Wire Wire Line
 	2050 5600 2250 5600
 Connection ~ 2250 5700
 Wire Wire Line
-	3000 5700 4600 5700
+	3000 5700 3700 5700
 Connection ~ 3700 5700
 Wire Wire Line
-	2250 6900 4600 6900
+	2250 6900 3000 6900
 Connection ~ 3700 6900
 $Sheet
@@
 $EndSheet
 Wire Wire Line
-	3700 3750 6950 3750
+	3700 3750 4600 3750
 Connection ~ 4600 3750
 Wire Wire Line
 	7850 2150 8200 2150
+Wire Wire Line
+	3700 5400 3900 5400
+Wire Wire Line
+	4600 5000 5000 5000
+Wire Wire Line
+	3850 4900 5000 4900
+Wire Wire Line
+	3700 6600 3900 6600
+Wire Wire Line
+	4600 6200 5000 6200
+Wire Wire Line
+	3850 6100 5000 6100
+Wire Wire Line
+	3000 6900 3000 7000
+Wire Wire Line
+	3000 6900 3700 6900
+Wire Wire Line
+	3700 3450 3900 3450
+Wire Wire Line
+	4600 3050 5000 3050
+Wire Wire Line
+	3850 2950 5000 2950
+Wire Wire Line
+	6950 3750 6950 3900
+Wire Wire Line
+	2250 5700 2250 6900
+Wire Wire Line
+	3700 5700 4600 5700
+Wire Wire Line
+	3700 6900 4600 6900
+Wire Wire Line
+	4600 3750 6950 3750
 $EndSCHEMATC
