File: Motherboard/ANALOG_EXPANSION.kicad_sch (KiCad schematic)
At the start: 43 parts

Commit message: Schematic ready.  Going to clean up directory now.
Parts:
- C1, C10, C11, C12, C2, C3, C4, C5, C6, C7, C8, C9: footprint Capacitors_SMD:C_1206 -> Capacitor_SMD:C_1206_3216Metric
- R14, R15, R16, R2, R20, R21, R22, R23, R24, R25, R26, R27, R28, R29, R3, R30, R31, R32, R33, R34, R35, R36, R37, R4: footprint Resistors_SMD:R_1206 -> Resistor_SMD:R_1206_3216Metric
Changed lines of the file:
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@@
 			)
 		)
-		(property "Footprint" "Capacitors_SMD:C_1206"
+		(property "Footprint" "Capacitor_SMD:C_1206_3216Metric"
 			(at 58.42 63.1952 0)
 			(effects
@@
 			)
 		)
-		(property "Footprint" "Capacitors_SMD:C_1206"
+		(property "Footprint" "Capacitor_SMD:C_1206_3216Metric"
 			(at 58.42 50.4952 0)
 			(effects
@@
 			)
 		)
-		(property "Footprint" "Capacitors_SMD:C_1206"
+		(property "Footprint" "Capacitor_SMD:C_1206_3216Metric"
 			(at 58.42 42.8752 0)
 			(effects
@@
 			)
 		)
-		(property "Footprint" "Capacitors_SMD:C_1206"
+		(property "Footprint" "Capacitor_SMD:C_1206_3216Metric"
 			(at 125.73 63.1952 0)
 			(effects
@@
 			)
 		)
-		(property "Footprint" "Capacitors_SMD:C_1206"
+		(property "Footprint" "Capacitor_SMD:C_1206_3216Metric"
 			(at 125.73 50.4952 0)
 			(effects
@@
 			)
 		)
-		(property "Footprint" "Capacitors_SMD:C_1206"
+		(property "Footprint" "Capacitor_SMD:C_1206_3216Metric"
 			(at 125.73 42.8752 0)
 			(effects
@@
 			)
 		)
-		(property "Footprint" "Capacitors_SMD:C_1206"
+		(property "Footprint" "Capacitor_SMD:C_1206_3216Metric"
 			(at 193.04 63.1952 0)
 			(effects
@@
 			)
 		)
-		(property "Footprint" "Capacitors_SMD:C_1206"
+		(property "Footprint" "Capacitor_SMD:C_1206_3216Metric"
 			(at 193.04 50.4952 0)
 			(effects
@@
 			)
 		)
-		(property "Footprint" "Capacitors_SMD:C_1206"
+		(property "Footprint" "Capacitor_SMD:C_1206_3216Metric"
 			(at 193.04 42.8752 0)
 			(effects
@@
 			)
 		)
-		(property "Footprint" "Capacitors_SMD:C_1206"
+		(property "Footprint" "Capacitor_SMD:C_1206_3216Metric"
 			(at 260.35 63.1952 0)
 			(effects
@@
 			)
 		)
-		(property "Footprint" "Capacitors_SMD:C_1206"
+		(property "Footprint" "Capacitor_SMD:C_1206_3216Metric"
 			(at 260.35 50.4952 0)
 			(effects
@@
 			)
 		)
-		(property "Footprint" "Capacitors_SMD:C_1206"
+		(property "Footprint" "Capacitor_SMD:C_1206_3216Metric"
 			(at 260.35 42.8752 0)
 			(effects
@@
 			)
 		)
-		(property "Footprint" "Resistors_SMD:R_1206"
+		(property "Footprint" "Resistor_SMD:R_1206_3216Metric"
 			(at 57.15 116.332 90)
 			(effects
@@
 			)
 		)
-		(property "Footprint" "Resistors_SMD:R_1206"
+		(property "Footprint" "Resistor_SMD:R_1206_3216Metric"
 			(at 57.15 118.872 90)
 			(effects
@@
 			)
 		)
-		(property "Footprint" "Resistors_SMD:R_1206"
+		(property "Footprint" "Resistor_SMD:R_1206_3216Metric"
 			(at 57.15 121.412 90)
 			(effects
@@
 			)
 		)
-		(property "Footprint" "Resistors_SMD:R_1206"
+		(property "Footprint" "Resistor_SMD:R_1206_3216Metric"
 			(at 57.15 123.952 90)
 			(effects
@@
 			)
 		)
-		(property "Footprint" "Resistors_SMD:R_1206"
+		(property "Footprint" "Resistor_SMD:R_1206_3216Metric"
 			(at 57.15 126.492 90)
 			(effects
@@
 			)
 		)
-		(property "Footprint" "Resistors_SMD:R_1206"
+		(property "Footprint" "Resistor_SMD:R_1206_3216Metric"
 			(at 57.15 129.032 90)
 			(effects
@@
 			)
 		)
-		(property "Footprint" "Resistors_SMD:R_1206"
+		(property "Footprint" "Resistor_SMD:R_1206_3216Metric"
 			(at 116.84 116.332 90)
 			(effects
@@
 			)
 		)
-		(property "Footprint" "Resistors_SMD:R_1206"
+		(property "Footprint" "Resistor_SMD:R_1206_3216Metric"
 			(at 116.84 118.872 90)
 			(effects
@@
 			)
 		)
-		(property "Footprint" "Resistors_SMD:R_1206"
+		(property "Footprint" "Resistor_SMD:R_1206_3216Metric"
 			(at 116.84 121.412 90)
 			(effects
@@
 			)
 		)
-		(property "Footprint" "Resistors_SMD:R_1206"
+		(property "Footprint" "Resistor_SMD:R_1206_3216Metric"
 			(at 116.84 123.952 90)
 			(effects
@@
 			)
 		)
-		(property "Footprint" "Resistors_SMD:R_1206"
+		(property "Footprint" "Resistor_SMD:R_1206_3216Metric"
 			(at 116.84 126.492 90)
 			(effects
@@
 			)
 		)
-		(property "Footprint" "Resistors_SMD:R_1206"
+		(property "Footprint" "Resistor_SMD:R_1206_3216Metric"
 			(at 116.84 129.032 90)
 			(effects
@@
 			)
 		)
-		(property "Footprint" "Resistors_SMD:R_1206"
+		(property "Footprint" "Resistor_SMD:R_1206_3216Metric"
 			(at 196.85 104.902 90)
 			(effects
@@
 			)
 		)
-		(property "Footprint" "Resistors_SMD:R_1206"
+		(property "Footprint" "Resistor_SMD:R_1206_3216Metric"
 			(at 221.742 138.43 90)
 			(effects
@@
 			)
 		)
-		(property "Footprint" "Resistors_SMD:R_1206"
+		(property "Footprint" "Resistor_SMD:R_1206_3216Metric"
 			(at 200.152 138.43 90)
 			(effects
@@
 			)
 		)
-		(property "Footprint" "Resistors_SMD:R_1206"
+		(property "Footprint" "Resistor_SMD:R_1206_3216Metric"
 			(at 243.332 111.76 90)
 			(effects
@@
 			)
 		)
-		(property "Footprint" "Resistors_SMD:R_1206"
+		(property "Footprint" "Resistor_SMD:R_1206_3216Metric"
 			(at 196.85 131.572 90)
 			(effects
@@
 			)
 		)
-		(property "Footprint" "Resistors_SMD:R_1206"
+		(property "Footprint" "Resistor_SMD:R_1206_3216Metric"
 			(at 240.03 104.902 90)
 			(effects
@@
 			)
 		)
-		(property "Footprint" "Resistors_SMD:R_1206"
+		(property "Footprint" "Resistor_SMD:R_1206_3216Metric"
 			(at 240.03 131.572 90)
 			(effects
@@
 			)
 		)
-		(property "Footprint" "Resistors_SMD:R_1206"
+		(property "Footprint" "Resistor_SMD:R_1206_3216Metric"
 			(at 218.44 131.572 90)
 			(effects
@@
 			)
 		)
-		(property "Footprint" "Resistors_SMD:R_1206"
+		(property "Footprint" "Resistor_SMD:R_1206_3216Metric"
 			(at 221.742 111.76 90)
 			(effects
@@
 			)
 		)
-		(property "Footprint" "Resistors_SMD:R_1206"
+		(property "Footprint" "Resistor_SMD:R_1206_3216Metric"
 			(at 218.44 104.902 90)
 			(effects
@@
 			)
 		)
-		(property "Footprint" "Resistors_SMD:R_1206"
+		(property "Footprint" "Resistor_SMD:R_1206_3216Metric"
 			(at 243.332 138.43 90)
 			(effects
@@
 			)
 		)
-		(property "Footprint" "Resistors_SMD:R_1206"
+		(property "Footprint" "Resistor_SMD:R_1206_3216Metric"
 			(at 200.152 111.76 90)
 			(effects
