File: Motherboard/Smart Tank Motherboard.kicad_pcb (KiCad board)
At the start: 10 copper layers, 400.1 x 266.7 mm, 324 parts, among them Q1 MOSFET_N_(FDMA430NZ), Q10 MOSFET_N_(FDMA430NZ), Q11 MOSFET_P_(BS250FTA), Q12 MOSFET_N_(2N7002P,215), Q13 MOSFET_N_(2N7002P,215), Q14 MOSFET_N_(FDMA430NZ), Q15 MOSFET_P_(BS250FTA), Q16 MOSFET_N_(2N7002P,215), Q17 MOSFET_N_(2N7002P,215), Q18 MOSFET_N_(FDMA430NZ), Q19 MOSFET_P_(BS250FTA), Q2 MOSFET_N_(2N7002P,215), Q20 MOSFET_N_(2N7002P,215), Q21 MOSFET_N_(2N7002P,215), Q22 MOSFET_N_(FDMA430NZ), Q23 MOSFET_P_(BS250FTA), Q24 MOSFET_N_(2N7002P,215), Q25 MOSFET_N_(2N7002P,215), Q26 MOSFET_N_(FDMA430NZ), Q27 MOSFET_P_(BS250FTA), Q3 MOSFET_N_(2N7002P,215), Q4 MOSFET_P_(BS250FTA), Q5 MOSFET_N_(2N7002P,215), Q6 MOSFET_N_(2N7002P,215), Q7 MOSFET_N_(2N7002P,215), Q8 MOSFET_N_(2N7002P,215), Q9 MOSFET_N_(2N7002P,215), U1 LM358, U2 LM358

Commit message: Started cleaning out old parts from PCB.
Parts:
- removed C18, C22: 1uF, Capacitors_SMD:C_1206
- removed C19: 10uF, Capacitors_SMD:C_1206
- removed C47, C48, C49, C50, C51, C52, C53, C54, C55, C56, C57, C58: 47nF, Capacitors_SMD:C_1206
- removed CAP_TOGGLE_1, CAP_TOGGLE_2, CAP_TOGGLE_3, CAP_TOGGLE_4, CAP_TOGGLE_5, CAP_TOGGLE_6: NKK_TOGGLE_(G3T12AP), Smart_Tank:NKK_TOGGLE_(G3T12AP)
- removed D1, D11, D13, D2, D5, D7, D9: DIODE_(1N4148X-TP), Diodes_SMD:SOD-523
- removed D16, D17, D18, D19, D20, D21: D, Diodes_SMD:D_SOD-123
- removed IGN_RLY_1, IGN_RLY_2, IGN_RLY_3, IGN_RLY_4, IGN_RLY_5, IGN_RLY_6, RELAY_1, RELAY_2: OMRON_RELAY_(G6L-1F-DC24), Smart_Tank:OMRON_RELAY_1A_(G6L-1F-DC24)
- removed INPUT_SEL_1, INPUT_SEL_2, INPUT_SEL_3, PUMP_CONFIG_1, PUMP_CONFIG_2, PUMP_CONFIG_3, PUMP_CONFIG_4, PUMP_CONFIG_5, PUMP_CONFIG_6: CTS_DIP_SW_(219-6MST), Smart_Tank:CST_DIP_SW_6-POS_(219-6MST)
- removed PUMP_AMPS_1, PUMP_AMPS_2, PUMP_AMPS_4, PUMP_AMPS_5, PUMP_AMPS_6: LEM_CURRENT_(HLSR_32-P/SP33), Smart_Tank:LEM_CURRENT_(HLSR_32-P-SP33)
- removed PWR_SEL_1, PWR_SEL_2, PWR_SEL_3: CONN_01X03, Pin_Headers:Pin_Header_Straight_1x03
- removed PWR_SEL_4: CONN_01X03, Pin_Headers:Pin_Header_Straight_1x03_Pitch2.54mm
- removed Q11, Q15, Q19, Q23, Q27, Q4: MOSFET_P_(BS250FTA), TO_SOT_Packages_SMD:SOT-23
- removed Q13, Q17, Q21, Q25, Q5, Q6, Q7, Q9: MOSFET_N_(2N7002P,215), TO_SOT_Packages_SMD:SOT-23
- removed R1, R13, R3, R53, R54, R62, R63, R71, R72, R80, R81, R89, R90: 150, Resistors_SMD:R_1206
- removed R2, R4, R50, R51, R59, R60, R68, R69, R77, R78, R86, R87: 10k, Resistors_SMD:R_1206
- removed R38, R39, R40, R41, R42, R43: 499, Resistors_SMD:R_1206
- removed R44: 1M, Resistors_SMD:R_1206
- removed R45, R46: 15k, Resistors_SMD:R_1206
- removed TC_INPUTS1: CONN_01X04, Smart_Tank:PHX_TB_HDR_4_POS_STR_(1755752)
- removed TEMP_1, TEMP_2: TEMP_COND_(AD8497), Housings_SSOP:MSOP-8_3x3mm_Pitch0.65mm
- added CAL10: CONN_01x01, Smart_Tank:FEMALE_SPADE_QC_(TE_63969-1), F.Cu at (551.3, 244.9)
- added CAL11: CONN_01x01, Smart_Tank:FEMALE_SPADE_QC_(TE_63969-1), F.Cu at (584.6, 173.7)
- added CAL12: CONN_01x01, Smart_Tank:FEMALE_SPADE_QC_(TE_63969-1), F.Cu at (584.6, 179.5)
- added CAL2: CONN_01x01, Smart_Tank:FEMALE_SPADE_QC_(TE_63969-1), F.Cu at (589.6, 205.0)
- added CAL3: CONN_01x01, Smart_Tank:FEMALE_SPADE_QC_(TE_63969-1), F.Cu at (575.0, 240.7)
- added CAL4: CONN_01x01, Smart_Tank:FEMALE_SPADE_QC_(TE_63969-1), F.Cu at (575.0, 246.5)
- added CAL5: CONN_01x01, Smart_Tank:FEMALE_SPADE_QC_(TE_63969-1), F.Cu at (597.7, 240.7)
- added CAL6: CONN_01x01, Smart_Tank:FEMALE_SPADE_QC_(TE_63969-1), F.Cu at (597.7, 246.5)
- added CAL7: CONN_01x01, Smart_Tank:FEMALE_SPADE_QC_(TE_63969-1), F.Cu at (528.6, 239.0)
- added CAL8: CONN_01x01, Smart_Tank:FEMALE_SPADE_QC_(TE_63969-1), F.Cu at (528.6, 244.9)
- added CAL9: CONN_01x01, Smart_Tank:FEMALE_SPADE_QC_(TE_63969-1), F.Cu at (551.3, 239.0)
- added CTRL_SHUNT_1: SHUNT_(WSL40261L000FEA), Smart_Tank:SHUNT_(WSL40261L000FEA), F.Cu at (577.2, 212.8)
- added CTRL_SHUNT_2: SHUNT_(WSL40261L000FEA), Smart_Tank:SHUNT_(WSL40261L000FEA), F.Cu at (562.6, 248.5)
- added CTRL_SHUNT_3: SHUNT_(WSL40261L000FEA), Smart_Tank:SHUNT_(WSL40261L000FEA), F.Cu at (585.2, 248.5)
- added CTRL_SHUNT_4: SHUNT_(WSL40261L000FEA), Smart_Tank:SHUNT_(WSL40261L000FEA), F.Cu at (516.2, 246.8)
- added CTRL_SHUNT_5: SHUNT_(WSL40261L000FEA), Smart_Tank:SHUNT_(WSL40261L000FEA), F.Cu at (538.8, 246.8)
- added CTRL_SHUNT_6: SHUNT_(WSL40261L000FEA), Smart_Tank:SHUNT_(WSL40261L000FEA), F.Cu at (572.1, 181.5)
- added HMI_CONN1: CONN_02X05, Connector_IDC:IDC-Header_2x05_P2.54mm_Vertical, F.Cu at (526.1, 208.6)
- added PUMP_CONFIG1: SW_DIP_x12 (SDA12H1SBD), Smart_Tank:SW_DIP_SPSTx12_(SDA12H1SBD), F.Cu at (565.1, 219.4)
- added PUMP_SHUNT_1: SHUNT_(WSL40261L000FEA), Smart_Tank:SHUNT_(WSL40261L000FEA), F.Cu at (577.2, 223.8)
- added PUMP_SHUNT_2: SHUNT_(WSL40261L000FEA), Smart_Tank:SHUNT_(WSL40261L000FEA), F.Cu at (562.6, 259.5)
- added PUMP_SHUNT_3: SHUNT_(WSL40261L000FEA), Smart_Tank:SHUNT_(WSL40261L000FEA), F.Cu at (585.2, 259.5)
- added PUMP_SHUNT_4: SHUNT_(WSL40261L000FEA), Smart_Tank:SHUNT_(WSL40261L000FEA), F.Cu at (516.2, 257.8)
- added PUMP_SHUNT_5: SHUNT_(WSL40261L000FEA), Smart_Tank:SHUNT_(WSL40261L000FEA), F.Cu at (538.8, 257.8)
- added PUMP_SHUNT_6: SHUNT_(WSL40261L000FEA), Smart_Tank:SHUNT_(WSL40261L000FEA), F.Cu at (572.1, 192.5)
- added PWR_SEL1: CONN_01X03, Connector_PinHeader_2.54mm:PinHeader_1x03_P2.54mm_Vertical, F.Cu at (456.3, 129.3)
- added RS232_CONN1: CONN_02X05, Connector_IDC:IDC-Header_2x05_P2.54mm_Vertical, F.Cu at (538.1, 208.6)
- added RS485_CONN1: CONN_02X05, Connector_IDC:IDC-Header_2x05_P2.54mm_Vertical, F.Cu at (550.1, 208.6)
- added RST_SW1: SW_Push, Button_Switch_SMD:SW_SPST_Omron_B3FS-100xP, F.Cu at (531.1, 228.8)
- C1, C10, C11, C12, C2, C20, C21, C29, C3, C30, C33, C34, C37, C38, C4, C41, C42, C45, C46, C5, C6, C7, C8, C9: footprint Capacitors_SMD:C_1206 -> Capacitor_SMD:C_1206_3216Metric
- C13, C15, C27, C28, C31, C32, C35, C36, C39, C40, C43, C44: value 47nF -> 0.1nF; footprint Capacitors_SMD:C_1206 -> Capacitor_SMD:C_1206_3216Metric
- C14, C25: value 1uF -> 0.01uF; footprint Capacitors_SMD:C_1206 -> Capacitor_SMD:C_1206_3216Metric
- C16: footprint Capacitors_SMD:C_1206 -> Smart_Tank:CAP_EEEHD1C100AR
- C17, C24: value 0.1uF -> 0.01uF; footprint Capacitors_SMD:C_1206 -> Capacitor_SMD:C_1206_3216Metric
- C23, C26: value 10uF -> 0.01uF; footprint Capacitors_SMD:C_1206 -> Capacitor_SMD:C_1206_3216Metric
- CAN_CONN1: footprint Connect:IDC_Header_Straight_10pins -> Connector_IDC:IDC-Header_2x05_P2.54mm_Vertical
- CTRL_AMPS_1, CTRL_AMPS_2, CTRL_AMPS_3, CTRL_AMPS_4, CTRL_AMPS_5, CTRL_AMPS_6: value LEM_CURRENT_(HLSR_32-P/SP33) -> CURRENT_AMP_(INA240A3); footprint Smart_Tank:LEM_CURRENT_(HLSR_32-P-SP33) -> Package_SO:SOIC-8_3.9x4.9mm_P1.27mm
- D10, D12, D14, D15, D6, D8: footprint Diodes_SMD:SOD-123 -> Diode_SMD:D_SMA
- D3, D4: value DIODE_(1N4148X-TP) -> D; footprint Diodes_SMD:SOD-523 -> Diode_SMD:D_SMA
- EXPANSION_CONN1: footprint Connect:IDC_Header_Straight_50pins -> Connector_IDC:IDC-Header_2x25_P2.54mm_Vertical
- PUMP_AMPS_3: value LEM_CURRENT_(HLSR_32-P/SP33) -> CURRENT_AMP_(INA240A2); footprint Smart_Tank:LEM_CURRENT_(HLSR_32-P-SP33) -> Package_SO:SOIC-8_3.9x4.9mm_P1.27mm
- PUMP_V_CONN_1, PUMP_V_CONN_2, PUMP_V_CONN_3, PUMP_V_CONN_4, PUMP_V_CONN_5, PUMP_V_CONN_6: footprint Smart_Tank:PHNX_TB_SCREW_4_POS_(1729144) -> Smart_Tank:PHX_TB_HDR_4_POS_STR_(1755752)
- PWR_RLY_1, PWR_RLY_2, PWR_RLY_3, PWR_RLY_4, PWR_RLY_5, PWR_RLY_6: value TE_AUTO_RELAY_(1432795-1) -> CIT_AUTO_RELAY_(A21CSQ24VDC1.6)
- Q1, Q10, Q14, Q18, Q22, Q26: value MOSFET_N_(FDMA430NZ) -> MOSFET_N_(DMN61D8LQ-13); footprint Smart_Tank:MOSFET_N_(FDMA430NZ) -> Package_TO_SOT_SMD:SOT-23
- Q12, Q16, Q20, Q24, Q3, Q8: value MOSFET_N_(2N7002P,215) -> MOSFET_N_(ZVN3320FTA); footprint TO_SOT_Packages_SMD:SOT-23 -> Package_TO_SOT_SMD:SOT-23
- Q2: value MOSFET_N_(2N7002P,215) -> MOSFET_N_(DMN61D8LQ-13); footprint TO_SOT_Packages_SMD:SOT-23 -> Package_TO_SOT_SMD:SOT-23
- R10, R8, R9: value 10k -> 2k; footprint Resistors_SMD:R_1206 -> Resistor_SMD:R_1206_3216Metric
- R11, R12: value 150 -> 2k; footprint Resistors_SMD:R_1206 -> Resistor_SMD:R_1206_3216Metric
- R14: value 1M -> 10k; footprint Resistors_SMD:R_1206 -> Resistor_SMD:R_1206_3216Metric
- R15: value 15k -> 100k; footprint Resistors_SMD:R_1206 -> Resistor_SMD:R_1206_3216Metric
- R16: value 15k -> 10k; footprint Resistors_SMD:R_1206 -> Resistor_SMD:R_1206_3216Metric
- R17, R18, R19, R20, R21, R22, R23, R24, R25, R26, R27, R28, R29, R30, R31, R47, R48, R49, R5, R52, R55, R56, R57, R58, R6, R61, R64, R65, R66, R67, R7, R70, R73, R74, R75, R76, R79, R82, R83, R84, R85, R88, R91, R92, R93: footprint Resistors_SMD:R_1206 -> Resistor_SMD:R_1206_3216Metric
- R32, R34, R36: value 249 -> 100k; footprint Resistors_SMD:R_1206 -> Resistor_SMD:R_1206_3216Metric
- R33, R35, R37: value 249 -> 10k; footprint Resistors_SMD:R_1206 -> Resistor_SMD:R_1206_3216Metric
- RIO_PWR_CONN1: footprint Smart_Tank:MOLEX_2-PIN_CONN_(0039300020) -> Smart_Tank:PHNX_TB_SCREW_2_POS_(1729128)
- moved R14 397.5 mm to (505.8, 275.7)
- moved R15 397.5 mm to (505.8, 273.2)
- moved R16 397.5 mm to (505.8, 278.2)
- moved Q2 111.3 mm to (121.2, 223.1), turned to 0 degrees
- moved C16 31.5 mm to (93.3, 297.2)
- moved C24 1.36 mm to (116.9, 303.6)
- moved Q3 1.22 mm to (152.1, 238.2), turned to 180 degrees
- moved PUMP_V_CONN_4 0.90 mm to (326.7, 328.9)
- moved PUMP_V_CONN_2 0.87 mm to (204.8, 328.9)
- moved PUMP_V_CONN_3 0.86 mm to (265.7, 328.9)
- moved PUMP_V_CONN_5 0.84 mm to (387.6, 328.9)
- moved PUMP_V_CONN_6 0.84 mm to (448.6, 328.9)
- moved PUMP_V_CONN_1 0.84 mm to (143.8, 328.9)
- moved Q1 0.55 mm to (123.1, 114.3)
- renumbered AI36-41_CONN1 to FLOW_CONN1, AI42-47_CONN1 to PH_VOLT_CONN1, AI30-35_CONN1 to PRESSURE_CONN1
Connections:
- net AI10 renamed -S_CTRL_3
- net AI11 renamed -S_CTRL_4
- net AI12 renamed -S_CTRL_5
- net AI13 renamed -S_CTRL_6
- net AI8 renamed -S_CTRL_1
- net AI9 renamed -S_CTRL_2
- net Net-(CTRL_CONN_1-Pad1) renamed +S_CTRL_1
- net Net-(CTRL_CONN_2-Pad1) renamed +S_CTRL_2
- net Net-(CTRL_CONN_3-Pad1) renamed +S_CTRL_3
- net Net-(CTRL_CONN_4-Pad1) renamed +S_CTRL_4
- net Net-(CTRL_CONN_5-Pad1) renamed +S_CTRL_5
- net Net-(CTRL_CONN_6-Pad1) renamed +S_CTRL_6
- net Net-(RMC_CONN1-Pad105) renamed DIO30
- net Net-(RMC_CONN1-Pad117) renamed DIO29
- net Net-(RMC_CONN1-Pad123) renamed DIO28
- net Net-(RMC_CONN1-Pad135) renamed DIO27
- net Net-(RMC_CONN1-Pad141) renamed DIO26
- net Net-(RMC_CONN1-Pad99) renamed DIO31
- AO_CONN1 pad 1: Net-(AO_CONN1-Pad1) -> Net-(AO_CONN1-P1)
- AO_CONN1 pad 2: Net-(AO_CONN1-Pad2) -> Net-(AO_CONN1-P2)
- AO_CONN1 pad 3: Net-(AO_CONN1-Pad3) -> Net-(AO_CONN1-P3)
- AO_CONN1 pad 4: Net-(AO_CONN1-Pad4) -> Net-(AO_CONN1-P4)
- C13 pad 1: GND -> 3.3VDC
- C13 pad 2: 3.3VDC -> GND
- C14 pad 1: Net-(C14-Pad1) -> Net-(CAL2-Pin_1)
- C15 pad 1: GND -> 3.3VDC
- C15 pad 2: 3.3VDC -> GND
- C16 pad 1: Net-(C16-Pad1) -> Net-(AO_CONN1-P1)
- C16 pad 2: Net-(C14-Pad1) -> GND
- C17 pad 1: 5VDC -> Net-(CAL12-Pin_1)
- C20 pad 1: GND -> AI16
- C20 pad 2: AI16 -> GND
- C21 pad 1: GND -> AI22
- C21 pad 2: AI22 -> GND
- C23 pad 1: Net-(C23-Pad1) -> Net-(CAL4-Pin_1)
- C23 pad 2: Net-(C22-Pad1) -> GND
- C24 pad 1: 5VDC -> Net-(CAL6-Pin_1)
- C25 pad 1: GND -> Net-(CAL8-Pin_1)
- C25 pad 2: Net-(C23-Pad1) -> GND
- C26 pad 1: 5VDC -> Net-(CAL10-Pin_1)
- C27 pad 1: GND -> 3.3VDC
- C27 pad 2: 3.3VDC -> GND
- C28 pad 1: GND -> 3.3VDC
- C28 pad 2: 3.3VDC -> GND
- C29 pad 1: GND -> AI17
- C29 pad 2: AI17 -> GND
- C30 pad 1: GND -> AI23
- C30 pad 2: AI23 -> GND
- C31 pad 1: GND -> 3.3VDC
- C31 pad 2: 3.3VDC -> GND
- C32 pad 1: GND -> 3.3VDC
- C32 pad 2: 3.3VDC -> GND
- C33 pad 1: GND -> AI18
- C33 pad 2: AI18 -> GND
- C34 pad 1: GND -> AI24
- C34 pad 2: AI24 -> GND
- C35 pad 1: GND -> 3.3VDC
- C35 pad 2: 3.3VDC -> GND
- C36 pad 1: GND -> 3.3VDC
- C36 pad 2: 3.3VDC -> GND
- C37 pad 1: GND -> AI19
- C37 pad 2: AI19 -> GND
- C38 pad 1: GND -> AI25
- C38 pad 2: AI25 -> GND
- C39 pad 1: GND -> 3.3VDC
- C39 pad 2: 3.3VDC -> GND
- C40 pad 1: GND -> 3.3VDC
- C40 pad 2: 3.3VDC -> GND
- C41 pad 1: GND -> AI20
- C41 pad 2: AI20 -> GND
- C42 pad 1: GND -> AI26
- C42 pad 2: AI26 -> GND
- C43 pad 1: GND -> 3.3VDC
- C43 pad 2: 3.3VDC -> GND
- C44 pad 1: GND -> 3.3VDC
- C44 pad 2: 3.3VDC -> GND
- C45 pad 1: GND -> AI21
- C45 pad 2: AI21 -> GND
- C46 pad 1: GND -> AI27
- C46 pad 2: AI27 -> GND
- CAN_CONN1 pad 1: Net-(CAN_CONN1-Pad1) -> unconnected-(CAN_CONN1-P1-Pad1)
- CAN_CONN1 pad 10: Net-(CAN_CONN1-Pad10) -> unconnected-(CAN_CONN1-P10-Pad10)
- CAN_CONN1 pad 4: Net-(CAN_CONN1-Pad4) -> unconnected-(CAN_CONN1-P4-Pad4)
- CAN_CONN1 pad 5: Net-(CAN_CONN1-Pad5) -> unconnected-(CAN_CONN1-P5-Pad5)
- CAN_CONN1 pad 6: Net-(CAN_CONN1-Pad6) -> unconnected-(CAN_CONN1-P6-Pad6)
- CAN_CONN1 pad 8: Net-(CAN_CONN1-Pad8) -> unconnected-(CAN_CONN1-P8-Pad8)
- CAN_CONN1 pad 9: Net-(CAN_CONN1-Pad9) -> unconnected-(CAN_CONN1-P9-Pad9)
- CTRL_AMPS_1 pad 2: AI22 -> GND
- CTRL_AMPS_1 pad 4: 3.3VDC -> unconnected-(CTRL_AMPS_1-NC-Pad4)
- CTRL_AMPS_1 pad 5: Net-(CTRL_AMPS_1-Pad5) -> AI22
- CTRL_AMPS_1 pad 6: Net-(CTRL_AMPS_1-Pad5) -> 3.3VDC
- CTRL_AMPS_1 pad 7: Net-(CTRL_AMPS_1-Pad5) -> GND
- CTRL_AMPS_1 pad 8: Net-(CTRL_AMPS_1-Pad10) -> Net-(CTRL_AMPS_1-IN+)
- CTRL_AMPS_2 pad 2: AI23 -> GND
- CTRL_AMPS_2 pad 4: 3.3VDC -> unconnected-(CTRL_AMPS_2-NC-Pad4)
- CTRL_AMPS_2 pad 5: Net-(CTRL_AMPS_2-Pad5) -> AI23
- CTRL_AMPS_2 pad 6: Net-(CTRL_AMPS_2-Pad5) -> 3.3VDC
- CTRL_AMPS_2 pad 7: Net-(CTRL_AMPS_2-Pad5) -> GND
- CTRL_AMPS_2 pad 8: Net-(CTRL_AMPS_2-Pad10) -> Net-(CTRL_AMPS_2-IN+)
- CTRL_AMPS_3 pad 2: AI24 -> GND
- CTRL_AMPS_3 pad 4: 3.3VDC -> unconnected-(CTRL_AMPS_3-NC-Pad4)
- CTRL_AMPS_3 pad 5: Net-(CTRL_AMPS_3-Pad5) -> AI24
- CTRL_AMPS_3 pad 6: Net-(CTRL_AMPS_3-Pad5) -> 3.3VDC
- CTRL_AMPS_3 pad 7: Net-(CTRL_AMPS_3-Pad5) -> GND
- CTRL_AMPS_3 pad 8: Net-(CTRL_AMPS_3-Pad10) -> Net-(CTRL_AMPS_3-IN+)
- CTRL_AMPS_4 pad 2: AI25 -> GND
- CTRL_AMPS_4 pad 4: 3.3VDC -> unconnected-(CTRL_AMPS_4-NC-Pad4)
- CTRL_AMPS_4 pad 5: Net-(CTRL_AMPS_4-Pad5) -> AI25
- CTRL_AMPS_4 pad 6: Net-(CTRL_AMPS_4-Pad5) -> 3.3VDC
- CTRL_AMPS_4 pad 7: Net-(CTRL_AMPS_4-Pad5) -> GND
- CTRL_AMPS_4 pad 8: Net-(CTRL_AMPS_4-Pad10) -> Net-(CTRL_AMPS_4-IN+)
- CTRL_AMPS_5 pad 2: AI26 -> GND
- CTRL_AMPS_5 pad 4: 3.3VDC -> unconnected-(CTRL_AMPS_5-NC-Pad4)
- CTRL_AMPS_5 pad 5: Net-(CTRL_AMPS_5-Pad5) -> AI26
- CTRL_AMPS_5 pad 6: Net-(CTRL_AMPS_5-Pad5) -> 3.3VDC
- CTRL_AMPS_5 pad 7: Net-(CTRL_AMPS_5-Pad5) -> GND
- CTRL_AMPS_5 pad 8: Net-(CTRL_AMPS_5-Pad10) -> Net-(CTRL_AMPS_5-IN+)
- CTRL_AMPS_6 pad 2: AI27 -> GND
- CTRL_AMPS_6 pad 4: 3.3VDC -> unconnected-(CTRL_AMPS_6-NC-Pad4)
- CTRL_AMPS_6 pad 5: Net-(CTRL_AMPS_6-Pad5) -> AI27
- CTRL_AMPS_6 pad 6: Net-(CTRL_AMPS_6-Pad5) -> 3.3VDC
- CTRL_AMPS_6 pad 7: Net-(CTRL_AMPS_6-Pad5) -> GND
- CTRL_AMPS_6 pad 8: Net-(CTRL_AMPS_6-Pad10) -> Net-(CTRL_AMPS_6-IN+)
- CTRL_CONN_1 pad 3: Net-(CTRL_CONN_1-Pad3) -> Net-(CTRL_CONN_1-PWM_CMD)
- CTRL_CONN_1 pad 4: POS_1_SPR_1 -> POS_1_DIAG
- CTRL_CONN_1 pad A1: Net-(CTRL_AMPS_1-Pad5) -> Net-(CTRL_CONN_1-V_BATT)
- CTRL_CONN_1 pad A6: Net-(CTRL_CONN_1-PadA6) -> POS_1_SPARE
- CTRL_CONN_2 pad 3: Net-(CTRL_CONN_2-Pad3) -> Net-(CTRL_CONN_2-PWM_CMD)
- CTRL_CONN_2 pad 4: POS_2_SPR_1 -> POS_2_DIAG
- CTRL_CONN_2 pad A1: Net-(CTRL_AMPS_2-Pad5) -> Net-(CTRL_CONN_2-V_BATT)
- CTRL_CONN_2 pad A6: Net-(CTRL_CONN_2-PadA6) -> POS_2_SPARE
- CTRL_CONN_3 pad 3: Net-(CTRL_CONN_3-Pad3) -> Net-(CTRL_CONN_3-PWM_CMD)
- CTRL_CONN_3 pad 4: POS_3_SPR_1 -> POS_3_DIAG
- CTRL_CONN_3 pad A1: Net-(CTRL_AMPS_3-Pad5) -> Net-(CTRL_CONN_3-V_BATT)
- CTRL_CONN_3 pad A3: Net-(CTRL_CONN_3-PadA3) -> Net-(CTRL_CONN_3-P1)
- CTRL_CONN_3 pad A6: Net-(CTRL_CONN_3-PadA6) -> POS_3_SPARE
- CTRL_CONN_4 pad 3: Net-(CTRL_CONN_4-Pad3) -> Net-(CTRL_CONN_4-PWM_CMD)
- CTRL_CONN_4 pad 4: POS_4_SPR_1 -> POS_4_DIAG
- CTRL_CONN_4 pad A1: Net-(CTRL_AMPS_4-Pad5) -> Net-(CTRL_CONN_4-V_BATT)
- CTRL_CONN_4 pad A6: Net-(CTRL_CONN_4-PadA6) -> POS_4_SPARE
- CTRL_CONN_5 pad 3: Net-(CTRL_CONN_5-Pad3) -> Net-(CTRL_CONN_5-PWM_CMD)
- CTRL_CONN_5 pad 4: POS_5_SPR_1 -> POS_5_DIAG
- CTRL_CONN_5 pad A1: Net-(CTRL_AMPS_5-Pad5) -> Net-(CTRL_CONN_5-V_BATT)
- CTRL_CONN_5 pad A6: Net-(CTRL_CONN_5-PadA6) -> POS_5_SPARE
- CTRL_CONN_6 pad 3: Net-(CTRL_CONN_6-Pad3) -> Net-(CTRL_CONN_6-PWM_CMD)
- CTRL_CONN_6 pad 4: POS_6_SPR_1 -> POS_6_DIAG
- CTRL_CONN_6 pad A1: Net-(CTRL_AMPS_6-Pad5) -> Net-(CTRL_CONN_6-V_BATT)
- CTRL_CONN_6 pad A6: Net-(CTRL_CONN_6-PadA6) -> POS_6_SPARE
- D10 pad 1: Net-(D10-Pad1) -> +S_PUMP_4
- D12 pad 1: Net-(D12-Pad1) -> +S_PUMP_5
- D14 pad 1: Net-(D14-Pad1) -> +S_PUMP_6
- D15 pad 1: Net-(D15-Pad1) -> +S_PUMP_1
- D3 pad 1: 24VDC -> Net-(CAL4-Pin_1)
- D3 pad 2: Net-(D3-Pad2) -> GND
- D4 pad 1: 24VDC -> Net-(CAL6-Pin_1)
- D4 pad 2: Net-(D4-Pad2) -> GND
- D6 pad 1: Net-(D6-Pad1) -> +S_PUMP_2
- D8 pad 1: Net-(D8-Pad1) -> +S_PUMP_3
- EXPANSION_CONN1 pad 13: Net-(EXPANSION_CONN1-Pad13) -> Net-(EXPANSION_CONN1-P13)
- EXPANSION_CONN1 pad 15: Net-(EXPANSION_CONN1-Pad15) -> Net-(EXPANSION_CONN1-P15)
- EXPANSION_CONN1 pad 17: Net-(EXPANSION_CONN1-Pad17) -> Net-(EXPANSION_CONN1-P17)
- EXPANSION_CONN1 pad 19: Net-(EXPANSION_CONN1-Pad19) -> Net-(EXPANSION_CONN1-P19)
- EXPANSION_CONN1 pad 21: Net-(EXPANSION_CONN1-Pad21) -> Net-(EXPANSION_CONN1-P21)
- EXPANSION_CONN1 pad 23: Net-(EXPANSION_CONN1-Pad23) -> Net-(EXPANSION_CONN1-P23)
- EXPANSION_CONN1 pad 25: Net-(EXPANSION_CONN1-Pad25) -> AI28
- EXPANSION_CONN1 pad 27: Net-(EXPANSION_CONN1-Pad27) -> AI29
- GPIO_CONN1 pad 1: Net-(GPIO_CONN1-Pad1) -> AI6
- GPIO_CONN1 pad 2: Net-(GPIO_CONN1-Pad2) -> AI14
- GPIO_CONN1 pad 3: Net-(GPIO_CONN1-Pad3) -> 485_A
- GPIO_CONN1 pad 4: Net-(GPIO_CONN1-Pad4) -> 485_B
- PUMP_AMPS_3 pad 2: AI18 -> GND
- PUMP_AMPS_3 pad 3: GND -> 3.3VDC
- PUMP_AMPS_3 pad 4: 3.3VDC -> unconnected-(PUMP_AMPS_3-NC-Pad4)
- PUMP_AMPS_3 pad 5: Net-(PUMP_AMPS_3-Pad5) -> AI18
- PUMP_AMPS_3 pad 6: Net-(PUMP_AMPS_3-Pad5) -> 3.3VDC
- PUMP_AMPS_3 pad 7: Net-(PUMP_AMPS_3-Pad5) -> GND
- PUMP_AMPS_3 pad 8: Net-(CTRL_CONN_3-PadA3) -> Net-(PUMP_AMPS_3-IN+)
- PUMP_CONN_1 pad 1: Net-(PUMP_AMPS_1-Pad5) -> Net-(CAL2-Pin_1)
- PUMP_CONN_2 pad 1: Net-(PUMP_AMPS_2-Pad5) -> Net-(CAL4-Pin_1)
- PUMP_CONN_3 pad 1: Net-(PUMP_AMPS_3-Pad5) -> Net-(CAL6-Pin_1)
- PUMP_CONN_4 pad 1: Net-(PUMP_AMPS_4-Pad5) -> Net-(CAL8-Pin_1)
- PUMP_CONN_5 pad 1: Net-(PUMP_AMPS_5-Pad5) -> Net-(CAL10-Pin_1)
- PUMP_CONN_6 pad 1: Net-(PUMP_AMPS_6-Pad5) -> Net-(CAL12-Pin_1)
- PUMP_FUSE_1 pad 6: Net-(CAP_TOGGLE_1-Pad6) -> Net-(PUMP_PWR_CONN_1-P1)
- PUMP_FUSE_1 pad 7: Net-(CAP_TOGGLE_1-Pad6) -> Net-(PUMP_PWR_CONN_1-P1)
- PUMP_FUSE_2 pad 6: Net-(CAP_TOGGLE_2-Pad6) -> Net-(PUMP_PWR_CONN_2-P1)
- PUMP_FUSE_2 pad 7: Net-(CAP_TOGGLE_2-Pad6) -> Net-(PUMP_PWR_CONN_2-P1)
- PUMP_FUSE_3 pad 6: Net-(CAP_TOGGLE_3-Pad6) -> Net-(PUMP_PWR_CONN_3-P1)
- PUMP_FUSE_3 pad 7: Net-(CAP_TOGGLE_3-Pad6) -> Net-(PUMP_PWR_CONN_3-P1)
- PUMP_FUSE_4 pad 6: Net-(CAP_TOGGLE_4-Pad6) -> Net-(PUMP_PWR_CONN_4-P1)
- PUMP_FUSE_4 pad 7: Net-(CAP_TOGGLE_4-Pad6) -> Net-(PUMP_PWR_CONN_4-P1)
- PUMP_FUSE_5 pad 6: Net-(CAP_TOGGLE_5-Pad6) -> Net-(PUMP_PWR_CONN_5-P1)
- PUMP_FUSE_5 pad 7: Net-(CAP_TOGGLE_5-Pad6) -> Net-(PUMP_PWR_CONN_5-P1)
- PUMP_FUSE_6 pad 6: Net-(CAP_TOGGLE_6-Pad6) -> Net-(PUMP_PWR_CONN_6-P1)
- PUMP_FUSE_6 pad 7: Net-(CAP_TOGGLE_6-Pad6) -> Net-(PUMP_PWR_CONN_6-P1)
- PUMP_PWR_CONN_1 pad 1: Net-(CAP_TOGGLE_1-Pad5) -> Net-(PUMP_PWR_CONN_1-P1)
- PUMP_PWR_CONN_2 pad 1: Net-(CAP_TOGGLE_2-Pad5) -> Net-(PUMP_PWR_CONN_2-P1)
- PUMP_PWR_CONN_3 pad 1: Net-(CAP_TOGGLE_3-Pad5) -> Net-(PUMP_PWR_CONN_3-P1)
- PUMP_PWR_CONN_4 pad 1: Net-(CAP_TOGGLE_4-Pad5) -> Net-(PUMP_PWR_CONN_4-P1)
- PUMP_PWR_CONN_5 pad 1: Net-(CAP_TOGGLE_5-Pad5) -> Net-(PUMP_PWR_CONN_5-P1)
- PUMP_PWR_CONN_6 pad 1: Net-(CAP_TOGGLE_6-Pad5) -> Net-(PUMP_PWR_CONN_6-P1)
- PUMP_V_CONN_1 pad 2: Net-(PUMP_CONFIG_1-Pad11) -> -S_PUMP_1
- PUMP_V_CONN_1 pad 3: POS_1_SPR_1 -> POS_1_DIAG
- PUMP_V_CONN_1 pad 4: POS_1_SPR_2 -> Net-(CTRL_CONN_1-PWM_CMD)
- PUMP_V_CONN_2 pad 2: Net-(PUMP_CONFIG_2-Pad11) -> -S_PUMP_2
- PUMP_V_CONN_2 pad 3: POS_2_SPR_1 -> POS_2_DIAG
- PUMP_V_CONN_2 pad 4: POS_2_SPR_2 -> Net-(CTRL_CONN_2-PWM_CMD)
- PUMP_V_CONN_3 pad 2: Net-(PUMP_CONFIG_3-Pad11) -> -S_PUMP_3
- PUMP_V_CONN_3 pad 3: POS_3_SPR_1 -> POS_3_DIAG
- PUMP_V_CONN_3 pad 4: POS_3_SPR_2 -> Net-(CTRL_CONN_3-PWM_CMD)
- PUMP_V_CONN_4 pad 2: Net-(PUMP_CONFIG_4-Pad11) -> -S_PUMP_4
- PUMP_V_CONN_4 pad 3: POS_4_SPR_1 -> POS_4_DIAG
- PUMP_V_CONN_4 pad 4: POS_4_SPR_2 -> Net-(CTRL_CONN_4-PWM_CMD)
- PUMP_V_CONN_5 pad 2: Net-(PUMP_CONFIG_5-Pad11) -> -S_PUMP_5
- PUMP_V_CONN_5 pad 3: POS_5_SPR_1 -> POS_5_DIAG
- PUMP_V_CONN_5 pad 4: POS_5_SPR_2 -> Net-(CTRL_CONN_5-PWM_CMD)
- PUMP_V_CONN_6 pad 2: Net-(PUMP_CONFIG_6-Pad11) -> -S_PUMP_6
- PUMP_V_CONN_6 pad 3: POS_6_SPR_1 -> POS_6_DIAG
- PUMP_V_CONN_6 pad 4: POS_6_SPR_2 -> Net-(CTRL_CONN_6-PWM_CMD)
- PWR_RLY_1 pad 30: Net-(CAP_TOGGLE_1-Pad6) -> Net-(PUMP_PWR_CONN_1-P1)
- PWR_RLY_1 pad 85: Net-(PWR_RLY_1-Pad85) -> Net-(PWR_RLY_1-C-)
- PWR_RLY_1 pad 87: Net-(CTRL_AMPS_1-Pad10) -> Net-(PWR_RLY_1-NO)
- PWR_RLY_1 pad 87a: Net-(PWR_RLY_1-Pad87a) -> unconnected-(PWR_RLY_1-NC-Pad87a)
- PWR_RLY_2 pad 30: Net-(CAP_TOGGLE_2-Pad6) -> Net-(PUMP_PWR_CONN_2-P1)
- PWR_RLY_2 pad 85: Net-(PWR_RLY_2-Pad85) -> Net-(PWR_RLY_2-C-)
- PWR_RLY_2 pad 87: Net-(CTRL_AMPS_2-Pad10) -> Net-(CAL3-Pin_1)
- PWR_RLY_2 pad 87a: Net-(PWR_RLY_2-Pad87a) -> unconnected-(PWR_RLY_2-NC-Pad87a)
- PWR_RLY_3 pad 30: Net-(CAP_TOGGLE_3-Pad6) -> Net-(PUMP_PWR_CONN_3-P1)
- PWR_RLY_3 pad 85: Net-(PWR_RLY_3-Pad85) -> Net-(PWR_RLY_3-C-)
- PWR_RLY_3 pad 87: Net-(CTRL_AMPS_3-Pad10) -> Net-(CAL5-Pin_1)
- PWR_RLY_3 pad 87a: Net-(PWR_RLY_3-Pad87a) -> unconnected-(PWR_RLY_3-NC-Pad87a)
- PWR_RLY_4 pad 30: Net-(CAP_TOGGLE_4-Pad6) -> Net-(PUMP_PWR_CONN_4-P1)
- PWR_RLY_4 pad 85: Net-(PWR_RLY_4-Pad85) -> Net-(PWR_RLY_4-C-)
- PWR_RLY_4 pad 87: Net-(CTRL_AMPS_4-Pad10) -> Net-(CAL7-Pin_1)
- PWR_RLY_4 pad 87a: Net-(PWR_RLY_4-Pad87a) -> unconnected-(PWR_RLY_4-NC-Pad87a)
- PWR_RLY_5 pad 30: Net-(CAP_TOGGLE_5-Pad6) -> Net-(PUMP_PWR_CONN_5-P1)
- PWR_RLY_5 pad 85: Net-(PWR_RLY_5-Pad85) -> Net-(PWR_RLY_5-C-)
- PWR_RLY_5 pad 87: Net-(CTRL_AMPS_5-Pad10) -> Net-(CAL9-Pin_1)
- PWR_RLY_5 pad 87a: Net-(PWR_RLY_5-Pad87a) -> unconnected-(PWR_RLY_5-NC-Pad87a)
- PWR_RLY_6 pad 30: Net-(CAP_TOGGLE_6-Pad6) -> Net-(PUMP_PWR_CONN_6-P1)
- PWR_RLY_6 pad 85: Net-(PWR_RLY_6-Pad85) -> Net-(PWR_RLY_6-C-)
- PWR_RLY_6 pad 87: Net-(CTRL_AMPS_6-Pad10) -> Net-(CAL11-Pin_1)
- PWR_RLY_6 pad 87a: Net-(PWR_RLY_6-Pad87a) -> unconnected-(PWR_RLY_6-NC-Pad87a)
- Q1 pad 1: Net-(PWR_RLY_1-Pad85) -> (no net)
- Q1 pad 2: Net-(PWR_RLY_1-Pad85) -> (no net)
- Q1 pad 3: Net-(Q1-Pad3) -> (no net)
- Q10 pad 1: Net-(PWR_RLY_2-Pad85) -> DIO7
- Q10 pad 2: Net-(PWR_RLY_2-Pad85) -> GND
- Q10 pad 3: Net-(Q10-Pad3) -> Net-(PWR_RLY_2-C-)
- Q12 pad 3: Net-(PUMP_CONFIG_3-Pad4) -> Net-(CTRL_CONN_3-PWM_CMD)
- Q14 pad 1: Net-(PWR_RLY_3-Pad85) -> DIO8
- Q14 pad 2: Net-(PWR_RLY_3-Pad85) -> GND
- Q14 pad 3: Net-(Q14-Pad3) -> Net-(PWR_RLY_3-C-)
- Q16 pad 3: Net-(PUMP_CONFIG_4-Pad4) -> Net-(CTRL_CONN_4-PWM_CMD)
- Q18 pad 1: Net-(PWR_RLY_4-Pad85) -> DIO9
- Q18 pad 2: Net-(PWR_RLY_4-Pad85) -> GND
- Q18 pad 3: Net-(Q18-Pad3) -> Net-(PWR_RLY_4-C-)
- Q2 pad 1: Net-(Q2-Pad1) -> (no net)
- Q2 pad 2: GND -> (no net)
- Q2 pad 3: Net-(D1-Pad2) -> (no net)
- Q20 pad 3: Net-(PUMP_CONFIG_5-Pad4) -> Net-(CTRL_CONN_5-PWM_CMD)
- Q22 pad 1: Net-(PWR_RLY_5-Pad85) -> DIO10
- Q22 pad 2: Net-(PWR_RLY_5-Pad85) -> GND
- Q22 pad 3: Net-(Q22-Pad3) -> Net-(PWR_RLY_5-C-)
- Q24 pad 3: Net-(PUMP_CONFIG_6-Pad4) -> Net-(CTRL_CONN_6-PWM_CMD)
- Q26 pad 1: Net-(PWR_RLY_6-Pad85) -> DIO11
- Q26 pad 2: Net-(PWR_RLY_6-Pad85) -> GND
- Q26 pad 3: Net-(Q26-Pad3) -> Net-(PWR_RLY_6-C-)
- Q3 pad 1: Net-(Q3-Pad1) -> Net-(Q8-G)
- Q3 pad 3: Net-(PUMP_CONFIG_1-Pad4) -> Net-(CTRL_CONN_2-PWM_CMD)
- Q8 pad 1: Net-(Q8-Pad1) -> Net-(Q8-G)
- Q8 pad 3: Net-(PUMP_CONFIG_2-Pad4) -> Net-(CTRL_CONN_2-PWM_CMD)
- R10 pad 1: GND -> POS_4_DIAG
- R10 pad 2: DIO21 -> 3.3VDC
- R11 pad 1: Net-(Q5-Pad1) -> POS_5_DIAG
- R11 pad 2: DIO18 -> 3.3VDC
- R12 pad 1: Net-(Q6-Pad1) -> POS_6_DIAG
- R12 pad 2: DIO20 -> 3.3VDC
- R14 pad 1: Net-(R14-Pad1) -> GND
- R14 pad 2: GND -> AI43
- R15 pad 1: Net-(R14-Pad1) -> Net-(PH_VOLT_CONN1-P8)
- R15 pad 2: Net-(C14-Pad1) -> AI44
- R16 pad 1: Net-(R16-Pad1) -> GND
- R16 pad 2: Net-(C16-Pad1) -> AI44
- R20 pad 2: Net-(INPUT_SEL_2-Pad12) -> AI36
- R21 pad 2: Net-(INPUT_SEL_2-Pad11) -> AI37
- R22 pad 2: Net-(INPUT_SEL_2-Pad10) -> AI38
- R23 pad 2: Net-(INPUT_SEL_2-Pad9) -> AI39
- R24 pad 2: Net-(INPUT_SEL_2-Pad8) -> AI40
- R25 pad 2: Net-(INPUT_SEL_2-Pad7) -> AI41
- R26 pad 2: Net-(INPUT_SEL_1-Pad12) -> AI30
- R27 pad 2: Net-(INPUT_SEL_1-Pad11) -> AI31
- R28 pad 2: Net-(INPUT_SEL_1-Pad10) -> AI32
- R29 pad 2: Net-(INPUT_SEL_1-Pad9) -> AI33
- R30 pad 2: Net-(INPUT_SEL_1-Pad8) -> AI34
- R31 pad 2: Net-(INPUT_SEL_1-Pad7) -> AI35
- R32 pad 1: GND -> Net-(PH_VOLT_CONN1-P5)
- R32 pad 2: Net-(INPUT_SEL_3-Pad12) -> AI47
- R33 pad 2: Net-(INPUT_SEL_3-Pad11) -> AI47
- R34 pad 1: GND -> Net-(PH_VOLT_CONN1-P6)
- R34 pad 2: Net-(INPUT_SEL_3-Pad10) -> AI46
- R35 pad 2: Net-(INPUT_SEL_3-Pad9) -> AI46
- R36 pad 1: GND -> Net-(PH_VOLT_CONN1-P7)
- R36 pad 2: Net-(INPUT_SEL_3-Pad8) -> AI45
- R37 pad 2: Net-(INPUT_SEL_3-Pad7) -> AI45
- R5 pad 1: Net-(Q3-Pad1) -> Net-(Q3-G)
- R52 pad 1: Net-(Q8-Pad1) -> Net-(Q8-G)
- R55 pad 1: Net-(PUMP_CONFIG_2-Pad4) -> Net-(CTRL_CONN_2-PWM_CMD)
- R55 pad 2: Net-(CTRL_AMPS_2-Pad10) -> Net-(CAL3-Pin_1)
- R64 pad 1: Net-(PUMP_CONFIG_3-Pad4) -> Net-(CTRL_CONN_3-PWM_CMD)
- R64 pad 2: Net-(CTRL_AMPS_3-Pad10) -> Net-(CAL5-Pin_1)
- R7 pad 1: Net-(PUMP_CONFIG_1-Pad4) -> Net-(CTRL_CONN_1-PWM_CMD)
- R7 pad 2: Net-(CTRL_AMPS_1-Pad10) -> Net-(PWR_RLY_1-NO)
- R73 pad 1: Net-(PUMP_CONFIG_4-Pad4) -> Net-(CTRL_CONN_4-PWM_CMD)
- R73 pad 2: Net-(CTRL_AMPS_4-Pad10) -> Net-(CAL7-Pin_1)
- R8 pad 1: GND -> POS_2_DIAG
- R8 pad 2: DIO18 -> 3.3VDC
- R82 pad 1: Net-(PUMP_CONFIG_5-Pad4) -> Net-(CTRL_CONN_5-PWM_CMD)
- R82 pad 2: Net-(CTRL_AMPS_5-Pad10) -> Net-(CAL9-Pin_1)
- R9 pad 1: GND -> POS_3_DIAG
- R9 pad 2: DIO20 -> 3.3VDC
- R91 pad 1: Net-(PUMP_CONFIG_6-Pad4) -> Net-(CTRL_CONN_6-PWM_CMD)
- R91 pad 2: Net-(CTRL_AMPS_6-Pad10) -> Net-(CAL11-Pin_1)
- RIO_AIO_CONN1 pad 28: Net-(RIO_AIO_CONN1-Pad28) -> Net-(RIO_AIO_CONN1-P28)
- RIO_AIO_CONN1 pad 30: Net-(RIO_AIO_CONN1-Pad30) -> Net-(RIO_AIO_CONN1-P30)
- RIO_AIO_CONN1 pad 32: Net-(RIO_AIO_CONN1-Pad32) -> Net-(RIO_AIO_CONN1-P32)
- RIO_AIO_CONN1 pad 34: Net-(RIO_AIO_CONN1-Pad34) -> Net-(RIO_AIO_CONN1-P34)
- RIO_AIO_CONN1 pad 36: Net-(RIO_AIO_CONN1-Pad36) -> unconnected-(RIO_AIO_CONN1-P36-Pad36)
- RIO_AIO_CONN1 pad 38: Net-(RIO_AIO_CONN1-Pad38) -> unconnected-(RIO_AIO_CONN1-P38-Pad38)
- RIO_AIO_CONN1 pad 40: Net-(RIO_AIO_CONN1-Pad40) -> unconnected-(RIO_AIO_CONN1-P40-Pad40)
- RIO_AIO_CONN1 pad 42: Net-(RIO_AIO_CONN1-Pad42) -> unconnected-(RIO_AIO_CONN1-P42-Pad42)
- RIO_AIO_CONN1 pad 44: Net-(RIO_AIO_CONN1-Pad44) -> unconnected-(RIO_AIO_CONN1-P44-Pad44)
- RIO_AIO_CONN1 pad 46: Net-(RIO_AIO_CONN1-Pad46) -> unconnected-(RIO_AIO_CONN1-P46-Pad46)
- RIO_AIO_CONN1 pad 48: Net-(RIO_AIO_CONN1-Pad48) -> unconnected-(RIO_AIO_CONN1-P48-Pad48)
- RIO_AIO_CONN1 pad 50: Net-(RIO_AIO_CONN1-Pad50) -> unconnected-(RIO_AIO_CONN1-P50-Pad50)
- RMC_CONN1 pad 104: Net-(RMC_CONN1-Pad104) -> unconnected-(RMC_CONN1-DIO62-Pad104)
- RMC_CONN1 pad 107: Net-(EXPANSION_CONN1-Pad27) -> Net-(EXPANSION_CONN1-P15)
- RMC_CONN1 pad 110: Net-(RMC_CONN1-Pad110) -> unconnected-(RMC_CONN1-DIO61-Pad110)
- RMC_CONN1 pad 113: Net-(EXPANSION_CONN1-Pad25) -> Net-(EXPANSION_CONN1-P13)
- RMC_CONN1 pad 125: Net-(EXPANSION_CONN1-Pad23) -> POS_6_DIAG
- RMC_CONN1 pad 131: Net-(EXPANSION_CONN1-Pad21) -> POS_5_DIAG
- RMC_CONN1 pad 143: Net-(EXPANSION_CONN1-Pad19) -> POS_4_DIAG
- RMC_CONN1 pad 149: Net-(EXPANSION_CONN1-Pad17) -> POS_3_DIAG
- RMC_CONN1 pad 161: Net-(EXPANSION_CONN1-Pad15) -> POS_2_DIAG
- RMC_CONN1 pad 167: Net-(EXPANSION_CONN1-Pad13) -> POS_1_DIAG
- RMC_CONN1 pad 182: Net-(RMC_CONN1-Pad182) -> unconnected-(RMC_CONN1-DIO53-Pad182)
- RMC_CONN1 pad 194: Net-(RMC_CONN1-Pad194) -> unconnected-(RMC_CONN1-DIO52-Pad194)
- RMC_CONN1 pad 200: Net-(RMC_CONN1-Pad200) -> unconnected-(RMC_CONN1-DIO51-Pad200)
- RMC_CONN1 pad 212: Net-(RMC_CONN1-Pad212) -> unconnected-(RMC_CONN1-DIO50-Pad212)
- RMC_CONN1 pad 218: Net-(RMC_CONN1-Pad218) -> Net-(EXPANSION_CONN1-P23)
- RMC_CONN1 pad 230: Net-(RMC_CONN1-Pad230) -> Net-(EXPANSION_CONN1-P21)
- RMC_CONN1 pad 43: (no net) -> Net-(RMC_CONN1-RST)
- RMC_CONN1 pad 89: Net-(RMC_CONN1-Pad89) -> Net-(EXPANSION_CONN1-P19)
- RMC_CONN1 pad 92: Net-(RMC_CONN1-Pad92) -> unconnected-(RMC_CONN1-DIO63-Pad92)
- RMC_CONN1 pad 95: Net-(RMC_CONN1-Pad95) -> Net-(EXPANSION_CONN1-P17)
Routing:
- net (no net): track 0.08 -> 1836.9 mm
- net Net-(CAL8-Pin_1): track 0.00 -> 1021.3 mm
- net Net-(PUMP_AMPS_4-Pad5): track 1021.3 -> 0.00 mm
- net Net-(PUMP_AMPS_6-Pad5): track 993.7 -> 0.00 mm
- net Net-(CAL12-Pin_1): track 0.00 -> 993.7 mm
- net Net-(PUMP_AMPS_2-Pad5): track 961.9 -> 0.00 mm
- net Net-(PUMP_AMPS_1-Pad5): track 932.2 -> 0.00 mm
- net Net-(CAL2-Pin_1): track 0.00 -> 932.2 mm
- net Net-(CAL10-Pin_1): track 0.00 -> 908.4 mm
- net Net-(PUMP_AMPS_5-Pad5): track 908.4 -> 0.00 mm
- net Net-(PUMP_AMPS_3-Pad5): track 874.9 -> 0.00 mm
- net GND: track 1001.4 -> 184.6 mm, vias 88 -> 59
- net POS_6_DIAG: track 0.00 -> 484.7 mm, vias 0 -> 2
- net -S_CTRL_6: track 482.7 -> 0.00 mm, vias 2 -> 0
- net AI13: track 0.00 -> 480.0 mm, vias 0 -> 1
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Other:
- board text added: "SMART TANK PCB, V1.2 TI AUTOMOTIVE 11/25"
- board text removed: "+TEMP_1"
- board text removed: "+TEMP_2"
- board text removed: "-TEMP_1"
- board text removed: "-TEMP_2"
- board text removed: "24V"
- board text removed: "5V"
- board text removed: "CTRL V_SENSE - 6 OFF, 5 OFF PUMP V_SENSE - 6 ON, 5 ON N-CH PWM_CMD - 4 OFF, 3 ON P-CH PWM_CMD - 4 ON, 3 OFF"
- board text removed: "DIP ON = 4-20mA INPUT DIP OFF = 5V INPUT"
- board text removed: "SMART TANK PCB, V1.1 TI AUTOMOTIVE 7/17"
- board text removed: "USE T-TYPE TC"
