File: Motherboard/Smart Tank Motherboard.kicad_pcb (KiCad board)
At the start: 10 copper layers, 400.1 x 266.7 mm, 689 parts, among them Q1 MOSFET_N_(DMN61D8LQ-13), Q10 MOSFET_N_(DMN61D8LQ-13), Q12 MOSFET_N_(ZVN3320FTA), Q14 MOSFET_N_(DMN61D8LQ-13), Q16 MOSFET_N_(ZVN3320FTA), Q18 MOSFET_N_(DMN61D8LQ-13), Q2 MOSFET_N_(DMN61D8LQ-13), Q20 MOSFET_N_(ZVN3320FTA), Q22 MOSFET_N_(DMN61D8LQ-13), Q24 MOSFET_N_(ZVN3320FTA), Q26 MOSFET_N_(DMN61D8LQ-13), Q3 MOSFET_N_(ZVN3320FTA), Q8 MOSFET_N_(ZVN3320FTA), U1 LM358, U2 LM358

Commit message: Almost done with PCB.  Tying up a few loose ends.
Parts:
- moved HMI_CONN1 458.3 mm to (86.1, 310.2)
- moved RST_SW1 456.5 mm to (87.7, 120.0)
- moved RS232_CONN1 322.9 mm to (220.1, 213.4)
- moved RS485_CONN1 148.0 mm to (412.9, 220.2)
- moved C16 52.8 mm to (104.1, 251.0), turned to 0 degrees
- moved RIO_PWR_CONN1 39.7 mm to (335.3, 159.3), turned to 0 degrees
- renumbered PUMP_CONFIG1 to VOLT_SENSE1
Routing:
- net GND: track 176.3 -> 1516.1 mm, vias 58 -> 72
- net SPARE_1: track 0.00 -> 428.2 mm
- net SPARE_2: track 0.00 -> 422.8 mm
- net SPARE_3: track 0.89 -> 417.3 mm
- net SPARE_4: track 0.00 -> 412.0 mm
- net SPARE_5: track 0.00 -> 408.3 mm
- net SPARE_6: track 0.00 -> 403.6 mm
- net Net-(RMC_CONN1-RST): track 0.00 -> 377.1 mm, vias 0 -> 2
- net 485_B: track 0.00 -> 338.1 mm, vias 0 -> 1
- net 485_A: track 0.00 -> 337.2 mm, vias 0 -> 1
- net Net-(HMI_CONN1-P1): track 0.00 -> 220.0 mm
- net Net-(HMI_CONN1-P2): track 0.00 -> 219.0 mm
- net Net-(HMI_CONN1-P3): track 0.00 -> 218.7 mm
- net Net-(HMI_CONN1-P4): track 0.00 -> 218.5 mm
- net Net-(HMI_CONN1-P5): track 0.00 -> 218.0 mm
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Other:
- board text added: "+"
- board text added: "-"
- board text added: "1"
- board text added: "2"
- board text added: "24V"
- board text added: "3"
- board text added: "4"
- board text added: "5"
- board text added: "6"
- board text added: "AI14"
- board text added: "AI6"
- board text added: "CONTROLLER"
- board text added: "CONTROLLER CONN A1 - VBATT A2 - GND A3 - P1 A4 - P2 A5 - P3 A6 - SPARE_1 1 - SENSE+ 2 - SENSE- 3 - PWM_CMD 4 - DIAG 5 - SPARE_2 6 - CAN_HI 7 - CAN_LO"
- board text added: "FLOW"
- board text added: "PHASE VOLTAGE"
- board text added: "PRESS CMD"
- board text added: "PRESSURE"
- board text added: "PS_CMD"
- board text added: "PUMP"
- board text added: "RS485_A"
- board text added: "RS485_B"
- board text added: "SMART TANK PCB, V1.2 TI AUTOMOTIVE 12/25"
- board text removed: "*1A MAX"
- board text removed: "AO0"
- board text removed: "AO1"
- board text removed: "CONTROLLER CONN A1 - VBATT A2 - GND A3 - P1 A4 - P2 A5 - P3 A6 - IGN 1 - SENSE+ 2 - SENSE- 3 - PWM_CMD 4 - SPARE_1 5 - SPARE_2 6 - CAN_HI 7 - CAN_LO"
- board text removed: "PWM_CMD"
- board text removed: "RLY_1_IN*"
- board text removed: "RLY_1_OUT*"
- board text removed: "RLY_2_IN*"
- board text removed: "RLY_2_OUT*"
- board text removed: "SMART TANK PCB, V1.2 TI AUTOMOTIVE 11/25"
