File: Motherboard/Smart Tank Motherboard.kicad_pcb (KiCad board)
At the start: 10 copper layers, 400.1 x 266.7 mm, 689 parts, among them Q1 MOSFET_N_(DMN61D8LQ-13), Q10 MOSFET_N_(DMN61D8LQ-13), Q12 MOSFET_N_(ZVN3320FTA), Q14 MOSFET_N_(DMN61D8LQ-13), Q16 MOSFET_N_(ZVN3320FTA), Q18 MOSFET_N_(DMN61D8LQ-13), Q2 MOSFET_N_(DMN61D8LQ-13), Q20 MOSFET_N_(ZVN3320FTA), Q22 MOSFET_N_(DMN61D8LQ-13), Q24 MOSFET_N_(ZVN3320FTA), Q26 MOSFET_N_(DMN61D8LQ-13), Q3 MOSFET_N_(ZVN3320FTA), Q8 MOSFET_N_(ZVN3320FTA), U1 LM358, U2 LM358

Commit message: Capacitor part issues...
Made these changes...

Concerning C13, C15, C27, C28, C31, C32, C35, C36, C39, C40, C43, C44
The schematic is wrong, and the BOM is correct.  These should all be 0.1uF
Concerning C20, C21, C29, C30, C33, C34, C37, C38, C41, C42, C45, C46
The BOM is wrong, and the schematic is correct.  These should all be 4.7nF
Parts:
- C13, C15, C27, C28, C31, C32, C35, C36, C39, C40, C43, C44: value 0.1nF -> 0.1uF
