File: Motherboard/Smart Tank Motherboard.kicad_sch (KiCad schematic)
At the start: 6 parts, among them Q2 MOSFET_N_(DMN61D8LQ-13)

Commit message: Almost done with PCB.  Tying up a few loose ends.
Parts:
- renumbered PUMP_CONFIG1 to VOLT_SENSE1
Changed lines of the file:
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@@
 		(dnp no)
 		(fields_autoplaced yes)
-		(property "Reference" "PUMP_CONFIG1"
+		(property "Reference" "VOLT_SENSE1"
 			(at 219.71 96.52 0)
 			(effects
@@
 			(project ""
 				(path "/9bd0ace5-d8c1-442c-86d3-58cb44e43f85"
-					(reference "PUMP_CONFIG1")
+					(reference "VOLT_SENSE1")
 					(unit 1)
 				)
