File: Smart Tank Current Shunt/Smart Tank Current Shunt.kicad_pcb (KiCad board)
At the start: 6 copper layers, 27 x 49.2 mm, 80 parts, among them J1 CURRENT_SHUNT_INTERFACE

Commit message: Committing what appears to be a bunch of backup files.  Haven't touched this project in a while, so I'm going for it.
Other:
- net class Default removed
